File: frothfet-12ch/sender_input.kicad_sch (KiCad schematic)
At the start: 5 parts

Commit message: schematic looking clean.
Parts:
- R101: footprint Resistor_SMD:R_0805_2012Metric_Pad1.20x1.40mm_HandSolder -> Resistor_SMD:R_1206_3216Metric_Pad1.30x1.75mm_HandSolder; LCSC (none) -> C870575
- R105: value 19.8K 0.1% -> 20K 0.1%; LCSC (none) -> C469660
Changed lines of the file:
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@@
 			)
 		)
-		(property "Value" "19.8K 0.1%"
+		(property "Value" "20K 0.1%"
 			(at 179.07 119.38 0)
 			(effects
@@
 			)
 		)
-		(property "LCSC" ""
+		(property "LCSC" "C469660"
 			(at 176.53 118.11 0)
 			(effects
@@
 			)
 		)
-		(property "Footprint" "Resistor_SMD:R_0805_2012Metric_Pad1.20x1.40mm_HandSolder"
+		(property "Footprint" "Resistor_SMD:R_1206_3216Metric_Pad1.30x1.75mm_HandSolder"
 			(at 160.02 114.3 0)
 			(effects
@@
 			)
 		)
-		(property "LCSC" ""
-			(at 160.02 114.3 0)
-			(effects
+		(property "LCSC" "C870575"
+			(at 160.02 114.3 0)
+			(effects

Commit message: updated bom
Parts:
- INPUT2: LCSC (none) -> C5359600
Changed lines of the file:
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@@
+			)
+		)
+		(property "LCSC" "C5359600"
+			(at 142.24 106.68 0)
+			(effects
+				(font
+					(size 1.27 1.27)
+				)
+				(hide yes)
 			)
 		)

Commit message: just need to route it...
Other:
- company: (none) -> https://github.com/hoeken/frothfet
- title: (none) -> FrothFET 12CH
Changed lines of the file:
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@@
 	(generator_version "8.0")
 	(paper "A4")
+	(title_block
+		(title "FrothFET 12CH")
+		(date "2024-08-17")
+		(rev "D")
+		(company "https://github.com/hoeken/frothfet")
+	)
 	(junction
 		(at 193.04 106.68)

Commit message: changed senders to screw terminals
Parts:
- INPUT2: footprint Connector_JST:JST_PH_B3B-PH-K_1x03_P2.00mm_Vertical -> yarrboard:1x03 2.54mm RA Pluggable Terminal Block; LCSC C5359600 -> C2927504 and C2927484
Changed lines of the file:
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@@
 			)
 		)
-		(property "Footprint" "Connector_JST:JST_PH_B3B-PH-K_1x03_P2.00mm_Vertical"
+		(property "Footprint" "yarrboard:1x03 2.54mm RA Pluggable Terminal Block"
 			(at 142.24 106.68 0)
 			(effects
@@
 			)
 		)
-		(property "LCSC" "C5359600"
+		(property "LCSC" "C2927504 and C2927484"
 			(at 142.24 106.68 0)
 			(effects

Commit message: more pre-production tweaks
Parts:
- INPUT2: footprint yarrboard:1x03 2.54mm RA Pluggable Terminal Block -> Connector_Phoenix_MC:PhoenixContact_MC_1,5_3-G-3.5_1x03_P3.50mm_Horizontal; LCSC C2927504 and C2927484 -> C5188296 and C5188250
Changed lines of the file:
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@@
 			)
 		)
-		(property "Footprint" "yarrboard:1x03 2.54mm RA Pluggable Terminal Block"
+		(property "Footprint" "Connector_Phoenix_MC:PhoenixContact_MC_1,5_3-G-3.5_1x03_P3.50mm_Horizontal"
 			(at 142.24 106.68 0)
 			(effects
@@
 			)
 		)
-		(property "Description" "Generic connector, single row, 01x03, script generated (kicad-library-utils/schlib/autogen/connector/)"
+		(property "Description" "pluggable terminal block 3.5mm 1x03"
 			(at 142.24 106.68 0)
 			(effects
@@
 			)
 		)
-		(property "LCSC" "C2927504 and C2927484"
+		(property "LCSC" "C5188296 and C5188250"
 			(at 142.24 106.68 0)
 			(effects
