File: frothfet-12ch/mosfet.kicad_sch (KiCad schematic)
At the start: 20 parts, among them J1 Conn_01x01, Q1 2N7002, Q2 BC846, Q3 BC856, Q4 IPB110P06LM, U2 ACS725xLCTR-20AU

Commit message: schematic looking clean.
Parts:
- R7: value 300K -> 300K 0.1%; LCSC (none) -> C865386
- R8: value 22K -> 22K 0.1%
Changed lines of the file:
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@@
 			)
 		)
-		(property "Value" "300K"
+		(property "Value" "300K 0.1%"
 			(at 127 128.27 0)
 			(effects
@@
 			)
 		)
-		(property "LCSC" ""
+		(property "LCSC" "C865386"
 			(at 124.46 127 0)
 			(effects
@@
 			)
 		)
-		(property "Value" "22K"
+		(property "Value" "22K 0.1%"
 			(at 127 140.97 0)
 			(effects

Commit message: updated bom
Parts:
- C2: Mouser 08053C104KAT4A -> (none)
- D1: LCSC (none) -> C94868
- D2: LCSC (none) -> C454989
- D3: LCSC (none) -> C511401
- F1: LCSC (none) -> C3204220
- J1: LCSC (none) -> C481447
- Q1: LCSC (none) -> C916396
- Q2: LCSC (none) -> C3037601
- Q3: LCSC (none) -> C7429738
- Q4: LCSC (none) -> C435954
- R5: LCSC (none) -> C114533
- R6: LCSC (none) -> C60816
Changed lines of the file:
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@@
+			)
+		)
+		(property "LCSC" "C511401"
+			(at 139.7 148.59 0)
+			(effects
+				(font
+					(size 1.27 1.27)
+				)
+				(hide yes)
 			)
 		)
@@
 			)
 		)
+		(property "LCSC" "C3037601"
+			(at 120.65 60.96 0)
+			(effects
+				(font
+					(size 1.27 1.27)
+				)
+				(hide yes)
+			)
+		)
 		(pin "1"
 		)
@@
 			)
 		)
+		(property "LCSC" "C114533"
+			(at 102.87 59.69 0)
+			(effects
+				(font
+					(size 1.27 1.27)
+				)
+				(hide yes)
+			)
+		)
 		(pin "1"
 		)
@@
 		)
 		(property "Mouser" "534-3522-3 "
+			(at 165.1 68.58 0)
+			(effects
+				(font
+					(size 1.27 1.27)
+				)
+				(hide yes)
+			)
+		)
+		(property "LCSC" "C3204220"
 			(at 165.1 68.58 0)
 			(effects
@@
 			)
 		)
+		(property "LCSC" "C94868"
+			(at 81.28 91.44 0)
+			(effects
+				(font
+					(size 1.27 1.27)
+				)
+				(hide yes)
+			)
+		)
 		(pin "1"
 		)
@@
 			)
 		)
-		(property "Mouser" "08053C104KAT4A"
+		(property "Mouser" ""
 			(at 166.37 102.87 0)
 			(effects
@@
 		)
 		(property "Description" ""
+			(at 102.87 71.12 0)
+			(effects
+				(font
+					(size 1.27 1.27)
+				)
+				(hide yes)
+			)
+		)
+		(property "LCSC" "C60816"
 			(at 102.87 71.12 0)
 			(effects
@@
 			)
 		)
+		(property "LCSC" "C7429738"
+			(at 120.65 71.12 0)
+			(effects
+				(font
+					(size 1.27 1.27)
+				)
+				(hide yes)
+			)
+		)
 		(pin "1"
 		)
@@
 			)
 		)
+		(property "LCSC" "C454989"
+			(at 93.98 59.69 0)
+			(effects
+				(font
+					(size 1.27 1.27)
+				)
+				(hide yes)
+			)
+		)
 		(pin "1"
 		)
@@
 			)
 		)
+		(property "LCSC" "C435954"
+			(at 137.16 66.04 0)
+			(effects
+				(font
+					(size 1.27 1.27)
+				)
+				(hide yes)
+			)
+		)
 		(pin "1"
 		)
@@
 			)
 		)
+		(property "LCSC" "C916396"
+			(at 100.33 81.28 0)
+			(effects
+				(font
+					(size 1.27 1.27)
+				)
+				(hide yes)
+			)
+		)
 		(pin "1"
 		)
@@
 			(at 162.56 143.51 0)
 			(effects
+				(font
+					(size 1.27 1.27)
+				)
+				(hide yes)
+			)
+		)
+		(property "LCSC" "C481447"
+			(at 162.56 143.51 0)
+			(effects

Commit message: just need to route it...
Other:
- company: https://github.com/hoeken/yarrboard -> https://github.com/hoeken/frothfet
- title: Yarrboard 8ch Mosfet Driver -> FrothFET 12CH
Changed lines of the file:
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@@
 	(paper "A4")
 	(title_block
-		(title "Yarrboard 8ch Mosfet Driver")
-		(rev "C1")
-		(company "https://github.com/hoeken/yarrboard")
+		(title "FrothFET 12CH")
+		(date "2024-08-17")
+		(rev "D")
+		(company "https://github.com/hoeken/frothfet")
 	)
 	(junction

Commit message: erc clean
Parts:
- F1: value 25A -> ATC Fuse Bypass; footprint yarrboard:ATC Bypass Fuse -> (none); symbol gnarboard:ATC Fuse Bypass -> yarrboard:ATC Fuse Bypass; LCSC C3204220 -> (none); Mouser 534-3522-3 -> (none)
- Q1: LCSC C916396 -> (none)
- Q4: footprint Package_TO_SOT_SMD:TO-263-2 -> Package_TO_SOT_THT:TO-220-3_Vertical; LCSC C435954 -> (none)
Changed lines of the file:
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@@
 	)
 	(symbol
-		(lib_id "gnarboard:ATC Fuse Bypass")
+		(lib_id "yarrboard:ATC Fuse Bypass")
 		(at 165.1 68.58 0)
 		(unit 1)
@@
 			)
 		)
-		(property "Value" "25A"
-			(at 157.48 64.77 0)
-			(effects
-				(font
-					(size 1.27 1.27)
-				)
-				(justify left)
-			)
-		)
-		(property "Footprint" "yarrboard:ATC Bypass Fuse"
-			(at 162.052 64.77 90)
+		(property "Value" "ATC Fuse Bypass"
+			(at 163.195 63.5 90)
+			(effects
+				(font
+					(size 1.27 1.27)
+				)
+			)
+		)
+		(property "Footprint" ""
+			(at 163.322 63.5 90)
 			(effects
 				(font
@@
 		)
 		(property "Datasheet" "~"
-			(at 163.83 64.77 0)
-			(effects
-				(font
-					(size 1.27 1.27)
-				)
-				(hide yes)
-			)
-		)
-		(property "Description" ""
-			(at 165.1 68.58 0)
-			(effects
-				(font
-					(size 1.27 1.27)
-				)
-				(hide yes)
-			)
-		)
-		(property "Mouser" "534-3522-3 "
-			(at 165.1 68.58 0)
-			(effects
-				(font
-					(size 1.27 1.27)
-				)
-				(hide yes)
-			)
-		)
-		(property "LCSC" "C3204220"
+			(at 165.1 63.5 0)
+			(effects
+				(font
+					(size 1.27 1.27)
+				)
+				(hide yes)
+			)
+		)
+		(property "Description" "Fuse"
 			(at 165.1 68.58 0)
 			(effects
@@
 			)
 		)
-		(property "Description" ""
+		(property "Description" "Power symbol creates a global label with name \"GNDPWR\" , global ground"
 			(at 139.7 158.75 0)
 			(effects
@@
 			)
 		)
-		(property "Footprint" "Package_TO_SOT_SMD:TO-263-2"
+		(property "Footprint" "Package_TO_SOT_THT:TO-220-3_Vertical"
 			(at 142.24 64.135 0)
 			(effects
@@
 			)
 		)
-		(property "Description" ""
-			(at 137.16 66.04 0)
-			(effects
-				(font
-					(size 1.27 1.27)
-				)
-				(hide yes)
-			)
-		)
-		(property "LCSC" "C435954"
+		(property "Description" "-74A Id, -55V Vds, Single P-Channel HEXFET Power MOSFET, 20mOhm Ron, TO-220AB"
 			(at 137.16 66.04 0)
 			(effects
@@
 			)
 		)
-		(property "Description" ""
+		(property "Description" "Power symbol creates a global label with name \"+24V\""
 			(at 168.91 46.99 0)
 			(effects
@@
 			)
 		)
-		(property "Description" ""
+		(property "Description" "Power symbol creates a global label with name \"GNDD\" , digital ground"
 			(at 93.98 97.79 0)
 			(effects
@@
 			)
 		)
-		(property "Description" ""
-			(at 100.33 81.28 0)
-			(effects
-				(font
-					(size 1.27 1.27)
-				)
-				(hide yes)
-			)
-		)
-		(property "LCSC" "C916396"
+		(property "Description" "0.115A Id, 60V Vds, N-Channel MOSFET, SOT-23"
 			(at 100.33 81.28 0)
 			(effects
@@
 			)
 		)
-		(property "Description" ""
+		(property "Description" "Power symbol creates a global label with name \"+3.3V\""
 			(at 149.86 101.6 0)
 			(effects
@@
 			)
 		)
-		(property "Description" ""
+		(property "Description" "Power symbol creates a global label with name \"GNDA\" , analog ground"
 			(at 149.86 125.73 0)
 			(effects

Commit message: just silkscreen and final review left.
Parts:
- Q4: footprint Package_TO_SOT_THT:TO-220-3_Vertical -> Package_TO_SOT_SMD:TO-263-2
Changed lines of the file:
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@@
 			)
 		)
-		(property "Footprint" "Package_TO_SOT_THT:TO-220-3_Vertical"
+		(property "Footprint" "Package_TO_SOT_SMD:TO-263-2"
 			(at 142.24 64.135 0)
 			(effects

Commit message: more pre-production tweaks
Parts:
- F1: footprint (none) -> yarrboard:ATC Bypass Fuse; Mouser (none) -> 534-3522-3
Changed lines of the file:
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@@
 			)
 		)
-		(property "Footprint" ""
+		(property "Footprint" "yarrboard:ATC Bypass Fuse"
 			(at 163.322 63.5 90)
 			(effects
@@
 			(at 165.1 68.58 0)
 			(effects
+				(font
+					(size 1.27 1.27)
+				)
+				(hide yes)
+			)
+		)
+		(property "Mouser" "534-3522-3 "
+			(at 165.1 68.58 0)
+			(effects

Commit message: added mosfet thermistor
Parts:
- added R112: 10K 0.1%, Resistor_SMD:R_0805_2012Metric_Pad1.20x1.40mm_HandSolder, symbol Device:R_Small_US
- added TH3: 10K, Resistor_SMD:R_0805_2012Metric_Pad1.20x1.40mm_HandSolder, symbol Device:Thermistor_NTC
Connections:
- net +3.3V: now also TH3.1
- net GNDA: now also R112.1
- new net THERMISTOR: R112.2, TH3.2
Other:
- note added: "Temperature Sensing"

Commit message: lots of big updates
Parts:
- removed D2: 15V, Diode_SMD:D_SOD-323_HandSoldering, symbol Device:D_Zener
- removed Q1: 2N7002, Package_TO_SOT_SMD:SOT-23, symbol Transistor_FET:2N7002
- removed Q2: BC846, Package_TO_SOT_SMD:SOT-23, symbol Transistor_BJT:BC846
- removed Q3: BC856, Package_TO_SOT_SMD:SOT-23, symbol Transistor_BJT:BC856
- removed Q4: IPB110P06LM, Package_TO_SOT_SMD:TO-263-2, symbol Transistor_FET:IRF4905
- removed R4: 220R, Resistor_SMD:R_0805_2012Metric_Pad1.20x1.40mm_HandSolder, symbol Device:R_Small_US
- removed R5: 27k, Resistor_SMD:R_0805_2012Metric_Pad1.20x1.40mm_HandSolder, symbol Device:R_Small_US
- removed R6: 4.7k, Resistor_SMD:R_0805_2012Metric_Pad1.20x1.40mm_HandSolder, symbol Device:R_Small_US
- removed TH3: 10K, Resistor_SMD:R_0805_2012Metric_Pad1.20x1.40mm_HandSolder, symbol Device:Thermistor_NTC
- added C62, C74: 100nF, Capacitor_SMD:C_0805_2012Metric_Pad1.18x1.45mm_HandSolder, symbol Device:C_Small
- added Q51: ISC011N06LM5ATMA1, yarrboard:Infineon_PG-TDSON-8_6.15x5.15mm, symbol Transistor_FET:IRF7480M
- added R124, R136: 0R, Resistor_SMD:R_0805_2012Metric_Pad1.20x1.40mm_HandSolder, symbol Device:R_Small_US
- added U23: LTC7003EMSE-TRPBF, 05-08-1667_ADI, symbol yarrboard:LTC7003EMSE-TRPBF
- D1: LCSC C94868 -> (none); Mouser 150080RS75000 -> (none)
- R112: value 10K 0.1% -> 0R; LCSC C110775 -> (none)
- renumbered R9 to R10, R7 to R8, R8 to R9
Connections:
- net GNDD is gone; now on net GNDPWR: D1.1 (K)
- net THERMISTOR is gone; now on net GNDPWR: R112.2
- net GNDA: no longer R112.1
- net GNDPWR: now also C62.2, R124.2, R136.2, U23.17 (GND)
- net PWM: now also U23.7 (INP)
- net at F1.1: now also Q51.1 (D), U23.1 (RUN), U23.2 (VIN)
- net at U2.1 (IP+), U2.2 (IP+): now also Q51.3 (S)
- new net: R136.1, U23.8 (OVLO)
- new net: R124.1, U23.6 (TIMER)
- new net: R112.1, U23.4 (VCCUV)
- new net: Q51.2 (G), U23.11 (TGDN), U23.12 (TGUP)
- new net: C62.1, U23.15 (SNS-), U23.16 (SNS+), U23.3 (VCC)
- new net: C74.1, U23.14 (BST)
- new net: C74.2, U23.13 (TS)
- no-connect marks 0 -> 3
Other:
- note removed: "Temperature Sensing"
- moved on the sheet: F1
