File: frothfet-12ch/mosfet.kicad_sch (KiCad schematic)
At the start: 19 parts, among them J1 Conn_01x01, Q51 ISC011N06LM5ATMA1, U2 ACS725xLCTR-20AU, U23 LTC7003EMSE-TRPBF

Commit message: changed to MIC5014
Parts:
- removed C62, C74: 100nF, Capacitor_SMD:C_0805_2012Metric_Pad1.18x1.45mm_HandSolder, symbol Device:C_Small
- removed D1: LED, LED_SMD:LED_0805_2012Metric_Pad1.15x1.40mm_HandSolder, symbol Device:LED
- removed R112, R124, R136: 0R, Resistor_SMD:R_0805_2012Metric_Pad1.20x1.40mm_HandSolder, symbol Device:R_Small_US
- removed U23: LTC7003EMSE-TRPBF, 05-08-1667_ADI, symbol yarrboard:LTC7003EMSE-TRPBF
- added C28: 100nF, Capacitor_SMD:C_0805_2012Metric_Pad1.18x1.45mm_HandSolder, symbol Device:C_Small
- added C46: 1uF/50v, Capacitor_SMD:C_0805_2012Metric_Pad1.18x1.45mm_HandSolder, symbol Device:C_Small
- added D1: 1N5817, Diode_SMD:Nexperia_CFP3_SOD-123W, symbol Diode:1N5817
- added D13, D34: 1N4001, Diode_SMD:Nexperia_CFP3_SOD-123W, symbol Diode:1N4001
- added D42: LED, LED_SMD:LED_0603_1608Metric_Pad1.05x0.95mm_HandSolder, symbol Device:LED
- added U11: MIC5014YM-TR, Package_SO:SOIC-8_3.9x4.9mm_P1.27mm, symbol yarrboard:MIC5014YM-TR
Connections:
- net GNDPWR: now also U11.4 (GROUND)
- net PWM: now also R3.1, U11.2 (INPUT); no longer R3.2
- net at F1.1, Q51.1 (D): now also D1.2 (A), D34.2 (A)
- net at Q51.3 (S), U2.1 (IP+), U2.2 (IP+): now also C28.2, C46.2, D42.1 (K), U11.3 (SOURCE)
- net at Q51.2 (G): now also U11.5 (GATE)
- new net: C28.1, D1.1 (K), D13.1 (K), U11.1 (V+)
- new net: C46.1, D13.2 (A), D34.1 (K)
- new net: D42.2 (A), R3.2
- no-connect marks 3 -> 0

Commit message: first pass at ltc7004
Parts:
- removed C46: 1uF/50v, Capacitor_SMD:C_0805_2012Metric_Pad1.18x1.45mm_HandSolder, symbol Device:C_Small
- removed D1: 1N5817, Diode_SMD:Nexperia_CFP3_SOD-123W, symbol Diode:1N5817
- removed D13, D34: 1N4001, Diode_SMD:Nexperia_CFP3_SOD-123W, symbol Diode:1N4001
- removed D42: LED, LED_SMD:LED_0603_1608Metric_Pad1.05x0.95mm_HandSolder, symbol Device:LED
- removed R3: 1k, Resistor_SMD:R_0805_2012Metric_Pad1.20x1.40mm_HandSolder, symbol Device:R_Small_US
- removed U11: MIC5014YM-TR, Package_SO:SOIC-8_3.9x4.9mm_P1.27mm, symbol yarrboard:MIC5014YM-TR
- added C1: 10uF/35v, Capacitor_SMD:C_1206_3216Metric_Pad1.33x1.80mm_HandSolder, symbol Device:C_Small
- added C66: 100nF, Capacitor_SMD:C_0805_2012Metric_Pad1.18x1.45mm_HandSolder, symbol Device:C_Small
- added D50: LED, LED_SMD:LED_0805_2012Metric_Pad1.15x1.40mm_HandSolder, symbol Device:LED
- added R47: 1k, Resistor_SMD:R_0805_2012Metric_Pad1.20x1.40mm_HandSolder, symbol Device:R_Small_US
- added R55, R63: 0R, Resistor_SMD:R_0805_2012Metric_Pad1.20x1.40mm_HandSolder, symbol Device:R_Small_US
- added U24: LTC7004EMSE-PBF, MSE_10_ADI, symbol yarrboard:LTC7004EMSE-PBF
- C2: renamed from C28; value 100nF -> 100nF/50v
- Q1: renamed from Q51; ALT (none) -> BSC010N04LS
- renumbered C1 to C4, C2 to C5, C3 to C6, D3 to D5, R8 to R4, R9 to R5, R10 to R6, U2 to U3
Connections:
- net GNDPWR: now also C2.2, C1.2, D50.1 (K), U24.2 (VCCUV), U24.3 (GND), U24.5 (OVLO), U24.EPAD
- net PWM: now also R47.1, U24.4 (INP)
- net +5V: now reaches C2.1
- net +5V: now also C1.1, U24.1 (VCC)
- net at Q1.3 (S), U3.1 (IP+), U3.2 (IP+): now also C66.2, U24.8 (TS); no longer C2.2
- net at Q1.2 (G): now also R55.1, R63.1
- new net: R63.2, U24.6 (TGDN)
- new net: R55.2, U24.7 (TGUP)
- new net: C66.1, U24.9 (BST)
- new net: D50.2 (A), R47.2
Other:
- note added: "Load Driver Circuit"
- note removed: "PWM MOSFET Channel"
- title: FrothFET 12CH -> FrothFET 8CH
- moved on the sheet: C2, C4, C5, C6, D5, F1, J1, Q1, R4, R5, R6, U3
