File: frothfet-12ch/adc.kicad_sch (KiCad schematic)
At the start: 4 parts, among them U10 MCP3564R

Commit message: first pass at ltc7004
Parts:
- renumbered C25 to C49, C26 to C50, C27 to C51, U10 to U18
Other:
- title: FrothFET 12CH -> FrothFET 8CH
Changed lines of the file:
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@@
 	(paper "A4")
 	(title_block
-		(title "FrothFET 12CH")
-		(date "2024-08-17")
+		(title "FrothFET 8CH")
+		(date "2024-08-21")
 		(rev "D")
 		(company "https://github.com/hoeken/frothfet")
@@
 		(on_board yes)
 		(dnp no)
-		(property "Reference" "C26"
+		(property "Reference" "C50"
 			(at 97.79 87.6363 0)
 			(effects
@@
 			(project ""
 				(path "/c83c6236-96e9-46ad-9d7a-9e2efa4a7966/b87f80e1-ecbd-4ee0-be26-4b252158928b"
-					(reference "C26")
+					(reference "C50")
 					(unit 1)
 				)
@@
 		(dnp no)
 		(fields_autoplaced yes)
-		(property "Reference" "#PWR072"
+		(property "Reference" "#PWR056"
 			(at 156.21 67.31 0)
 			(effects
@@
 			(project ""
 				(path "/c83c6236-96e9-46ad-9d7a-9e2efa4a7966/b87f80e1-ecbd-4ee0-be26-4b252158928b"
-					(reference "#PWR072")
+					(reference "#PWR056")
 					(unit 1)
 				)
@@
 		(on_board yes)
 		(dnp no)
-		(property "Reference" "#PWR070"
+		(property "Reference" "#PWR054"
 			(at 137.16 116.84 0)
 			(effects
@@
 			(project ""
 				(path "/c83c6236-96e9-46ad-9d7a-9e2efa4a7966/b87f80e1-ecbd-4ee0-be26-4b252158928b"
-					(reference "#PWR070")
+					(reference "#PWR054")
 					(unit 1)
 				)
@@
 		(dnp no)
 		(fields_autoplaced yes)
-		(property "Reference" "#PWR071"
+		(property "Reference" "#PWR055"
 			(at 144.78 116.84 0)
 			(effects
@@
 			(project ""
 				(path "/c83c6236-96e9-46ad-9d7a-9e2efa4a7966/b87f80e1-ecbd-4ee0-be26-4b252158928b"
-					(reference "#PWR071")
+					(reference "#PWR055")
 					(unit 1)
 				)
@@
 		(on_board yes)
 		(dnp no)
-		(property "Reference" "C25"
+		(property "Reference" "C49"
 			(at 87.63 87.6363 0)
 			(effects
@@
 			(project "frothfet-12ch"
 				(path "/c83c6236-96e9-46ad-9d7a-9e2efa4a7966/b87f80e1-ecbd-4ee0-be26-4b252158928b"
-					(reference "C25")
+					(reference "C49")
 					(unit 1)
 				)
@@
 		(on_board yes)
 		(dnp no)
-		(property "Reference" "C27"
+		(property "Reference" "C51"
 			(at 171.45 86.3663 0)
 			(effects
@@
 			(project ""
 				(path "/c83c6236-96e9-46ad-9d7a-9e2efa4a7966/b87f80e1-ecbd-4ee0-be26-4b252158928b"
-					(reference "C27")
+					(reference "C51")
 					(unit 1)
 				)
@@
 		(on_board yes)
 		(dnp no)
-		(property "Reference" "U10"
+		(property "Reference" "U18"
 			(at 120.396 71.12 0)
 			(effects
@@
 			(project ""
 				(path "/c83c6236-96e9-46ad-9d7a-9e2efa4a7966/b87f80e1-ecbd-4ee0-be26-4b252158928b"
-					(reference "U10")
+					(reference "U18")
 					(unit 1)
 				)
