File: frothfet-12ch/frothfet-12ch.kicad_sch (KiCad schematic)
At the start: 8 parts

Commit message: first pass at ltc7004
Other:
- title: FrothFET 12CH -> FrothFET 8CH
Changed lines of the file:
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@@
 	(paper "A4")
 	(title_block
-		(title "FrothFET 12CH")
-		(date "2024-08-17")
+		(title "FrothFET 8CH")
+		(date "2024-08-21")
 		(rev "D")
 		(company "https://github.com/hoeken/frothfet")
