File: frothfet-12ch/power.kicad_sch (KiCad schematic)
At the start: 32 parts, among them J10 Screw_Terminal_01x12, J9 Screw_Terminal_01x12, U11 MCP1502-33, U12 MCP3425A0T-ECH, U13 XL1509-5.0

Commit message: schematic looking clean.
Parts:
- added VREF1: SolderJumper_2_Open, Jumper:SolderJumper-2_P1.3mm_Open_RoundedPad1.0x1.5mm, symbol Jumper:SolderJumper_2_Open
- renumbered JP3 to 3V3
Connections:
- net REF_3V3: now also VREF1.2 (B); no longer R63.2, U11.1 (OUT)
- new net: R63.2, U11.1 (OUT), VREF1.1 (A)
Changed lines of the file:
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@@
 		(color 0 0 0 0)
 	)
+	(junction
+		(at 69.85 114.3)
+		(diameter 0)
+		(color 0 0 0 0)
+	)
 	(wire
 		(pts
@@
 	(wire
 		(pts
-			(xy 69.85 114.3) (xy 69.85 129.54)
-		)
-		(stroke
-			(width 0)
-			(type default)
-		)
-	)
-	(wire
-		(pts
 			(xy 30.48 48.26) (xy 30.48 49.53)
 		)
@@
 	(wire
 		(pts
-			(xy 69.85 129.54) (xy 72.39 129.54)
+			(xy 69.85 129.54) (xy 77.47 129.54)
 		)
 		(stroke
@@
 	(wire
 		(pts
+			(xy 77.47 114.3) (xy 77.47 129.54)
+		)
+		(stroke
+			(width 0)
+			(type default)
+		)
+	)
+	(wire
+		(pts
 			(xy 196.85 82.55) (xy 196.85 81.28)
 		)
@@
 	(wire
 		(pts
+			(xy 69.85 104.14) (xy 69.85 114.3)
+		)
+		(stroke
+			(width 0)
+			(type default)
+		)
+	)
+	(wire
+		(pts
 			(xy 234.95 127) (xy 238.76 127)
 		)
@@
 	(global_label "REF_3V3"
 		(shape input)
-		(at 72.39 129.54 0)
+		(at 69.85 104.14 0)
 		(fields_autoplaced yes)
 		(effects
@@
 		)
 		(property "Intersheetrefs" "${INTERSHEET_REFS}"
-			(at 83.358 129.54 0)
+			(at 80.818 104.14 0)
 			(effects
 				(font
@@
 		(on_board yes)
 		(dnp no)
-		(property "Reference" "JP3"
+		(property "Reference" "3V3"
 			(at 66.04 111.76 0)
 			(effects
@@
 			(project "8ch-mosfet"
 				(path "/c83c6236-96e9-46ad-9d7a-9e2efa4a7966/e112a34f-fd2f-43cb-bf5d-a7f5e57b6bef"
-					(reference "JP3")
+					(reference "3V3")
 					(unit 1)
 				)
@@
 					(unit 1)
 				)
+			)
+		)
+	)
+	(symbol
+		(lib_id "Jumper:SolderJumper_2_Open")
+		(at 73.66 114.3 180)
+		(unit 1)
+		(exclude_from_sim no)
+		(in_bom no)
+		(on_board yes)
+		(dnp no)
+		(property "Reference" "VREF1"
+			(at 73.66 111.76 0)
+			(effects
+				(font
+					(size 1.27 1.27)
+				)
+			)
+		)
+		(property "Value" "SolderJumper_2_Open"
+			(at 73.66 110.49 0)
+			(effects
+				(font
+					(size 1.27 1.27)
+				)
+				(hide yes)
+			)
+		)
+		(property "Footprint" "Jumper:SolderJumper-2_P1.3mm_Open_RoundedPad1.0x1.5mm"
+			(at 73.66 114.3 0)
+			(effects
+				(font
+					(size 1.27 1.27)
+				)
+				(hide yes)
+			)
+		)
+		(property "Datasheet" "~"
+			(at 73.66 114.3 0)
+			(effects
+				(font
+					(size 1.27 1.27)
+				)
+				(hide yes)
+			)
+		)
+		(property "Description" ""
+			(at 73.66 114.3 0)
+			(effects
+				(font
+					(size 1.27 1.27)
+				)
+				(hide yes)
+			)
+		)
+		(pin "1"
+		)
+		(pin "2"
+		)
+		(instances
+			(project "frothfet-12ch"
+				(path "/c83c6236-96e9-46ad-9d7a-9e2efa4a7966/e112a34f-fd2f-43cb-bf5d-a7f5e57b6bef"
+					(reference "VREF1")
+					(unit 1)
+				)

Commit message: updated bom
Parts:
- C26, C28, C31: Mouser 08053C104KAT4A -> (none)
- C27: LCSC (none) -> C83170
- C29: LCSC (none) -> C1952580
- C30: LCSC (none) -> C106843
- C32: value 1uF/50v -> 100nF; LCSC (none) -> C49678
- C33: LCSC (none) -> C2991173
- C34: value 22uF/35v -> 10uF/35v; footprint Capacitor_SMD:C_0805_2012Metric_Pad1.18x1.45mm_HandSolder -> Capacitor_SMD:C_1206_3216Metric_Pad1.33x1.80mm_HandSolder; LCSC (none) -> C454102
- D30, D33: value SX33L -> SS34; LCSC (none) -> C8678; Mouser 241-SX33L_R1_00001 -> 512-SS34
- R63: LCSC (none) -> C84376
- R66: LCSC (none) -> C137513
- U12: Mouser 579-MCP3425A0T-E/CH -> 579-MCP3425A0T-E/CH
Changed lines of the file:
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@@
 			)
 		)
-		(property "Value" "22uF/35v"
+		(property "Value" "10uF/35v"
 			(at 153.67 58.4263 0)
 			(effects
@@
 			)
 		)
-		(property "Footprint" "Capacitor_SMD:C_0805_2012Metric_Pad1.18x1.45mm_HandSolder"
+		(property "Footprint" "Capacitor_SMD:C_1206_3216Metric_Pad1.33x1.80mm_HandSolder"
 			(at 151.13 57.15 0)
 			(effects
@@
 			)
 		)
+		(property "LCSC" "C454102"
+			(at 151.13 57.15 0)
+			(effects
+				(font
+					(size 1.27 1.27)
+				)
+				(hide yes)
+			)
+		)
 		(pin "1"
 		)
@@
 			)
 		)
-		(property "Mouser" "08053C104KAT4A"
+		(property "Mouser" ""
 			(at 35.56 128.27 0)
 			(effects
@@
 			)
 		)
-		(property "Value" "SX33L"
+		(property "Value" "SS34"
 			(at 246.38 45.72 0)
 			(effects
@@
 			)
 		)
-		(property "Mouser" " 241-SX33L_R1_00001"
+		(property "Mouser" " 512-SS34 "
 			(at 246.38 49.53 90)
 			(effects
@@
 			)
 		)
+		(property "LCSC" "C8678"
+			(at 246.38 49.53 0)
+			(effects
+				(font
+					(size 1.27 1.27)
+				)
+				(hide yes)
+			)
+		)
 		(pin "1"
 		)
@@
 			)
 		)
+		(property "LCSC" "C84376"
+			(at 69.85 137.16 0)
+			(effects
+				(font
+					(size 1.27 1.27)
+				)
+				(hide yes)
+			)
+		)
 		(pin "1"
 		)
@@
 			)
 		)
-		(property "Value" "1uF/50v"
+		(property "Value" "100nF"
 			(at 124.46 58.4263 0)
 			(effects
@@
 			)
 		)
+		(property "LCSC" "C49678"
+			(at 121.92 57.15 0)
+			(effects
+				(font
+					(size 1.27 1.27)
+				)
+				(hide yes)
+			)
+		)
 		(pin "1"
 		)
@@
 			)
 		)
+		(property "LCSC" "C83170"
+			(at 68.58 57.15 0)
+			(effects
+				(font
+					(size 1.27 1.27)
+				)
+				(hide yes)
+			)
+		)
 		(pin "1"
 		)
@@
 			)
 		)
+		(property "LCSC" "C2991173"
+			(at 137.16 53.34 0)
+			(effects
+				(font
+					(size 1.27 1.27)
+				)
+				(hide yes)
+			)
+		)
 		(pin "1"
 		)
@@
 			)
 		)
+		(property "LCSC" "C137513"
+			(at 137.16 60.96 0)
+			(effects
+				(font
+					(size 1.27 1.27)
+				)
+				(hide yes)
+			)
+		)
 		(pin "1"
 		)
@@
 			)
 		)
-		(property "Mouser" "08053C104KAT4A"
+		(property "Mouser" ""
 			(at 102.87 132.08 0)
 			(effects
@@
 			)
 		)
-		(property "Mouser" " 579-MCP3425A0T-E/CH "
+		(property "Mouser" "579-MCP3425A0T-E/CH "
 			(at 157.48 132.08 0)
 			(effects
@@
 			)
 		)
-		(property "Value" "SX33L"
+		(property "Value" "SS34"
 			(at 93.98 45.72 0)
 			(effects
@@
 			)
 		)
-		(property "Mouser" " 241-SX33L_R1_00001"
+		(property "Mouser" " 512-SS34 "
 			(at 93.98 49.53 90)
 			(effects
@@
 			)
 		)
+		(property "LCSC" "C8678"
+			(at 93.98 49.53 0)
+			(effects
+				(font
+					(size 1.27 1.27)
+				)
+				(hide yes)
+			)
+		)
 		(pin "1"
 		)
@@
 			)
 		)
+		(property "LCSC" "C106843"
+			(at 102.87 57.15 0)
+			(effects
+				(font
+					(size 1.27 1.27)
+				)
+				(hide yes)
+			)
+		)
 		(pin "1"
 		)
@@
 			)
 		)
-		(property "Mouser" "08053C104KAT4A"
+		(property "Mouser" ""
 			(at 69.85 144.78 0)
 			(effects
@@
 			(at 93.98 132.08 0)
 			(effects
+				(font
+					(size 1.27 1.27)
+				)
+				(hide yes)
+			)
+		)
+		(property "LCSC" "C1952580"
+			(at 93.98 132.08 0)
+			(effects

Commit message: just need to route it...
Other:
- company: https://github.com/hoeken/yarrboard -> https://github.com/hoeken/frothfet
- title: Yarrboard 8ch Mosfet Driver -> FrothFET 12CH
Changed lines of the file:
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@@
 	(paper "A4")
 	(title_block
-		(title "Yarrboard 8ch Mosfet Driver")
-		(rev "C1")
-		(company "https://github.com/hoeken/yarrboard")
+		(title "FrothFET 12CH")
+		(date "2024-08-17")
+		(rev "D")
+		(company "https://github.com/hoeken/frothfet")
 	)
 	(junction

Commit message: erc clean
Changed lines of the file:
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@@
 	)
 	(junction
+		(at 69.85 109.22)
+		(diameter 0)
+		(color 0 0 0 0)
+	)
+	(junction
 		(at 213.36 49.53)
 		(diameter 0)
@@
 	(wire
 		(pts
+			(xy 69.85 109.22) (xy 69.85 114.3)
+		)
+		(stroke
+			(width 0)
+			(type default)
+		)
+	)
+	(wire
+		(pts
 			(xy 234.95 144.78) (xy 238.76 144.78)
 		)
@@
 	(wire
 		(pts
-			(xy 69.85 104.14) (xy 69.85 114.3)
+			(xy 69.85 100.33) (xy 69.85 109.22)
 		)
 		(stroke
@@
 	(global_label "REF_3V3"
 		(shape input)
-		(at 69.85 104.14 0)
+		(at 69.85 100.33 0)
 		(fields_autoplaced yes)
 		(effects
@@
 		)
 		(property "Intersheetrefs" "${INTERSHEET_REFS}"
-			(at 80.818 104.14 0)
+			(at 80.818 100.33 0)
 			(effects
 				(font
@@
 			)
 		)
-		(property "Description" ""
+		(property "Description" "Power symbol creates a global label with name \"+3.3V\""
 			(at 130.81 106.68 0)
 			(effects
@@
 			)
 		)
-		(property "Description" ""
+		(property "Description" "Power symbol creates a global label with name \"+3.3V\""
 			(at 62.23 113.03 0)
 			(effects
@@
 			)
 		)
-		(property "Description" ""
+		(property "Description" "Special symbol for telling ERC where power comes from"
 			(at 146.05 48.26 0)
 			(effects
@@
 			)
 		)
-		(property "Description" ""
+		(property "Description" "Special symbol for telling ERC where power comes from"
 			(at 256.54 49.53 0)
 			(effects
@@
 			)
 		)
-		(property "Description" ""
+		(property "Description" "Special symbol for telling ERC where power comes from"
 			(at 213.36 49.53 0)
 			(effects
@@
 			)
 		)
-		(property "Description" ""
+		(property "Description" "Special symbol for telling ERC where power comes from"
 			(at 30.48 48.26 0)
 			(effects
@@
 			)
 		)
-		(property "Description" ""
+		(property "Description" "Special symbol for telling ERC where power comes from"
 			(at 196.85 81.28 0)
 			(effects
@@
 			)
 		)
-		(property "Description" ""
+		(property "Description" "Special symbol for telling ERC where power comes from"
 			(at 154.94 81.28 0)
 			(effects
@@
 			)
 		)
-		(property "Description" ""
+		(property "Description" "Power symbol creates a global label with name \"+24V\""
 			(at 113.03 118.11 0)
 			(effects
@@
 			)
 		)
-		(property "Description" ""
+		(property "Description" "Power symbol creates a global label with name \"GNDA\" , analog ground"
 			(at 130.81 153.67 0)
 			(effects
@@
 	)
 	(symbol
+		(lib_id "power:PWR_FLAG")
+		(at 69.85 109.22 0)
+		(unit 1)
+		(exclude_from_sim no)
+		(in_bom yes)
+		(on_board yes)
+		(dnp no)
+		(property "Reference" "#FLG011"
+			(at 69.85 107.315 0)
+			(effects
+				(font
+					(size 1.27 1.27)
+				)
+				(hide yes)
+			)
+		)
+		(property "Value" "PWR_FLAG"
+			(at 69.85 104.14 0)
+			(effects
+				(font
+					(size 1.27 1.27)
+				)
+			)
+		)
+		(property "Footprint" ""
+			(at 69.85 109.22 0)
+			(effects
+				(font
+					(size 1.27 1.27)
+				)
+				(hide yes)
+			)
+		)
+		(property "Datasheet" "~"
+			(at 69.85 109.22 0)
+			(effects
+				(font
+					(size 1.27 1.27)
+				)
+				(hide yes)
+			)
+		)
+		(property "Description" "Special symbol for telling ERC where power comes from"
+			(at 69.85 109.22 0)
+			(effects
+				(font
+					(size 1.27 1.27)
+				)
+				(hide yes)
+			)
+		)
+		(pin "1"
+		)
+		(instances
+			(project "frothfet-12ch"
+				(path "/c83c6236-96e9-46ad-9d7a-9e2efa4a7966/e112a34f-fd2f-43cb-bf5d-a7f5e57b6bef"
+					(reference "#FLG011")
+					(unit 1)
+				)
+			)
+		)
+	)
+	(symbol
 		(lib_id "Device:R_Small_US")
 		(at 137.16 60.96 0)
@@
 			)
 		)
-		(property "Description" ""
+		(property "Description" "Power symbol creates a global label with name \"GNDPWR\" , global ground"
 			(at 238.76 153.67 0)
 			(effects
@@
 			)
 		)
-		(property "Description" ""
+		(property "Description" "Power symbol creates a global label with name \"+24V\""
 			(at 217.17 118.11 0)
 			(effects
@@
 			)
 		)
-		(property "Description" ""
+		(property "Description" "Power symbol creates a global label with name \"GNDPWR\" , global ground"
 			(at 154.94 82.55 0)
 			(effects
@@
 			)
 		)
-		(property "Description" ""
+		(property "Description" "Power symbol creates a global label with name \"GNDD\" , digital ground"
 			(at 176.53 82.55 0)
 			(effects
@@
 			)
 		)
-		(property "Description" ""
+		(property "Description" "Power symbol creates a global label with name \"+5V\""
 			(at 234.95 43.18 0)
 			(effects
@@
 			)
 		)
-		(property "Description" ""
+		(property "Description" "Power symbol creates a global label with name \"GNDA\" , analog ground"
 			(at 196.85 82.55 0)
 			(effects
@@
 			)
 		)
-		(property "Description" ""
+		(property "Description" "Power symbol creates a global label with name \"+24V\""
 			(at 30.48 35.56 0)
 			(effects
@@
 			)
 		)
-		(property "Description" ""
+		(property "Description" "Special symbol for telling ERC where power comes from"
 			(at 234.95 49.53 0)
 			(effects
@@
 			)
 		)
-		(property "Description" ""
+		(property "Description" "Power symbol creates a global label with name \"GNDA\" , analog ground"
 			(at 48.26 153.67 0)
 			(effects
@@
 			)
 		)
-		(property "Description" ""
+		(property "Description" "Special symbol for telling ERC where power comes from"
 			(at 76.2 48.26 0)
 			(effects
@@
 			)
 		)
-		(property "Description" ""
+		(property "Description" "Special symbol for telling ERC where power comes from"
 			(at 176.53 81.28 0)
 			(effects

Commit message: more pre-production tweaks
Parts:
- removed 3V3, VREF1: SolderJumper_2_Open, Jumper:SolderJumper-2_P1.3mm_Open_RoundedPad1.0x1.5mm, symbol Jumper:SolderJumper_2_Open
- added J15: Conn_01x03_Pin, Connector_PinHeader_2.54mm:PinHeader_1x03_P2.54mm_Vertical, symbol Connector:Conn_01x03_Pin
Connections:
- net +3.3V: now also J15.1 (Pin_1)
- net REF_3V3: now also J15.2 (Pin_2)
- net at R63.2, U11.1 (OUT): now also J15.3 (Pin_3)
Changed lines of the file:
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@@
 	)
 	(junction
-		(at 69.85 109.22)
-		(diameter 0)
-		(color 0 0 0 0)
-	)
-	(junction
 		(at 213.36 49.53)
 		(diameter 0)
@@
 		(color 0 0 0 0)
 	)
-	(junction
-		(at 69.85 114.3)
-		(diameter 0)
-		(color 0 0 0 0)
-	)
 	(wire
 		(pts
@@
 	(wire
 		(pts
+			(xy 77.47 111.76) (xy 77.47 129.54)
+		)
+		(stroke
+			(width 0)
+			(type default)
+		)
+	)
+	(wire
+		(pts
 			(xy 170.18 81.28) (xy 170.18 83.82)
 		)
@@
 	(wire
 		(pts
+			(xy 69.85 105.41) (xy 69.85 111.76)
+		)
+		(stroke
+			(width 0)
+			(type default)
+		)
+	)
+	(wire
+		(pts
 			(xy 213.36 121.92) (xy 217.17 121.92)
 		)
@@
 	(wire
 		(pts
-			(xy 62.23 114.3) (xy 62.23 113.03)
+			(xy 58.42 111.76) (xy 58.42 110.49)
 		)
 		(stroke
@@
 	(wire
 		(pts
-			(xy 69.85 109.22) (xy 69.85 114.3)
-		)
-		(stroke
-			(width 0)
-			(type default)
-		)
-	)
-	(wire
-		(pts
 			(xy 234.95 144.78) (xy 238.76 144.78)
 		)
@@
 	(wire
 		(pts
+			(xy 58.42 111.76) (xy 67.31 111.76)
+		)
+		(stroke
+			(width 0)
+			(type default)
+		)
+	)
+	(wire
+		(pts
 			(xy 69.85 139.7) (xy 69.85 142.24)
 		)
@@
 	(wire
 		(pts
-			(xy 57.15 120.65) (xy 57.15 121.92)
+			(xy 72.39 111.76) (xy 77.47 111.76)
 		)
 		(stroke
@@
 	(wire
 		(pts
-			(xy 44.45 120.65) (xy 44.45 129.54)
+			(xy 57.15 120.65) (xy 57.15 121.92)
 		)
 		(stroke
@@
 	(wire
 		(pts
-			(xy 238.76 132.08) (xy 238.76 129.54)
+			(xy 44.45 120.65) (xy 44.45 129.54)
 		)
 		(stroke
@@
 	(wire
 		(pts
-			(xy 234.95 59.69) (xy 234.95 66.04)
+			(xy 238.76 132.08) (xy 238.76 129.54)
 		)
 		(stroke
@@
 	(wire
 		(pts
-			(xy 93.98 109.22) (xy 102.87 109.22)
+			(xy 234.95 59.69) (xy 234.95 66.04)
 		)
 		(stroke
@@
 	(wire
 		(pts
-			(xy 213.36 49.53) (xy 223.52 49.53)
+			(xy 93.98 109.22) (xy 102.87 109.22)
 		)
 		(stroke
@@
 	(wire
 		(pts
-			(xy 238.76 127) (xy 238.76 124.46)
+			(xy 213.36 49.53) (xy 223.52 49.53)
 		)
 		(stroke
@@
 	(wire
 		(pts
-			(xy 77.47 114.3) (xy 77.47 129.54)
+			(xy 238.76 127) (xy 238.76 124.46)
 		)
 		(stroke
@@
 	(wire
 		(pts
-			(xy 69.85 100.33) (xy 69.85 109.22)
-		)
-		(stroke
-			(width 0)
-			(type default)
-		)
-	)
-	(wire
-		(pts
 			(xy 234.95 127) (xy 238.76 127)
 		)
@@
 	(global_label "REF_3V3"
 		(shape input)
-		(at 69.85 100.33 0)
+		(at 69.85 105.41 0)
 		(fields_autoplaced yes)
 		(effects
@@
 		)
 		(property "Intersheetrefs" "${INTERSHEET_REFS}"
-			(at 80.818 100.33 0)
+			(at 80.818 105.41 0)
 			(effects
 				(font
@@
 	(symbol
 		(lib_id "power:+3.3V")
-		(at 62.23 113.03 0)
+		(at 58.42 110.49 0)
 		(unit 1)
 		(exclude_from_sim no)
@@
 		(fields_autoplaced yes)
 		(property "Reference" "#PWR059"
-			(at 62.23 116.84 0)
+			(at 58.42 114.3 0)
 			(effects
 				(font
@@
 		)
 		(property "Value" "+3.3V"
-			(at 62.23 107.95 0)
+			(at 58.42 105.41 0)
 			(effects
 				(font
@@
 		)
 		(property "Footprint" ""
-			(at 62.23 113.03 0)
+			(at 58.42 110.49 0)
 			(effects
 				(font
@@
 		)
 		(property "Datasheet" ""
-			(at 62.23 113.03 0)
+			(at 58.42 110.49 0)
 			(effects
 				(font
@@
 		)
 		(property "Description" "Power symbol creates a global label with name \"+3.3V\""
-			(at 62.23 113.03 0)
+			(at 58.42 110.49 0)
 			(effects
 				(font
@@
 	)
 	(symbol
-		(lib_id "Jumper:SolderJumper_2_Open")
-		(at 66.04 114.3 180)
-		(unit 1)
-		(exclude_from_sim no)
-		(in_bom no)
-		(on_board yes)
-		(dnp no)
-		(property "Reference" "3V3"
-			(at 66.04 111.76 0)
-			(effects
-				(font
-					(size 1.27 1.27)
-				)
-			)
-		)
-		(property "Value" "SolderJumper_2_Open"
-			(at 66.04 110.49 0)
-			(effects
-				(font
-					(size 1.27 1.27)
-				)
-				(hide yes)
-			)
-		)
-		(property "Footprint" "Jumper:SolderJumper-2_P1.3mm_Open_RoundedPad1.0x1.5mm"
-			(at 66.04 114.3 0)
-			(effects
-				(font
-					(size 1.27 1.27)
-				)
-				(hide yes)
-			)
-		)
-		(property "Datasheet" "~"
-			(at 66.04 114.3 0)
-			(effects
-				(font
-					(size 1.27 1.27)
-				)
-				(hide yes)
-			)
-		)
-		(property "Description" ""
-			(at 66.04 114.3 0)
-			(effects
-				(font
-					(size 1.27 1.27)
-				)
-				(hide yes)
-			)
-		)
-		(pin "1"
-		)
-		(pin "2"
-		)
-		(instances
-			(project "8ch-mosfet"
-				(path "/c83c6236-96e9-46ad-9d7a-9e2efa4a7966/e112a34f-fd2f-43cb-bf5d-a7f5e57b6bef"
-					(reference "3V3")
-					(unit 1)
-				)
-			)
-		)
-	)
-	(symbol
 		(lib_id "power:PWR_FLAG")
 		(at 213.36 49.53 0)
@@
 	)
 	(symbol
-		(lib_id "Jumper:SolderJumper_2_Open")
-		(at 73.66 114.3 180)
+		(lib_id "Connector:Conn_01x03_Pin")
+		(at 69.85 116.84 90)
 		(unit 1)
 		(exclude_from_sim no)
-		(in_bom no)
+		(in_bom yes)
 		(on_board yes)
 		(dnp no)
-		(property "Reference" "VREF1"
-			(at 73.66 111.76 0)
+		(property "Reference" "J15"
+			(at 69.596 117.856 90)
 			(effects
 				(font
@@
 			)
 		)
-		(property "Value" "SolderJumper_2_Open"
-			(at 73.66 110.49 0)
+		(property "Value" "Conn_01x03_Pin"
+			(at 69.85 121.92 90)
 			(effects
 				(font
@@
 			)
 		)
-		(property "Footprint" "Jumper:SolderJumper-2_P1.3mm_Open_RoundedPad1.0x1.5mm"
-			(at 73.66 114.3 0)
+		(property "Footprint" "Connector_PinHeader_2.54mm:PinHeader_1x03_P2.54mm_Vertical"
+			(at 69.85 116.84 0)
 			(effects
 				(font
@@
 		)
 		(property "Datasheet" "~"
-			(at 73.66 114.3 0)
+			(at 69.85 116.84 0)
 			(effects
 				(font
@@
 			)
 		)
-		(property "Description" ""
-			(at 73.66 114.3 0)
+		(property "Description" "Generic connector, single row, 01x03, script generated"
+			(at 69.85 116.84 0)
 			(effects
 				(font
@@
 			)
 		)
-		(pin "1"
-		)
 		(pin "2"
 		)
+		(pin "3"
+		)
+		(pin "1"
+		)
 		(instances
-			(project "frothfet-12ch"
+			(project ""
 				(path "/c83c6236-96e9-46ad-9d7a-9e2efa4a7966/e112a34f-fd2f-43cb-bf5d-a7f5e57b6bef"
-					(reference "VREF1")
+					(reference "J15")
 					(unit 1)
 				)
@@
 	(symbol
 		(lib_id "power:PWR_FLAG")
-		(at 69.85 109.22 0)
+		(at 69.85 105.41 0)
 		(unit 1)
 		(exclude_from_sim no)
@@
 		(dnp no)
 		(property "Reference" "#FLG011"
-			(at 69.85 107.315 0)
+			(at 69.85 103.505 0)
 			(effects
 				(font
@@
 		)
 		(property "Value" "PWR_FLAG"
-			(at 69.85 104.14 0)
+			(at 69.85 100.33 0)
 			(effects
 				(font
@@
 		)
 		(property "Footprint" ""
-			(at 69.85 109.22 0)
+			(at 69.85 105.41 0)
 			(effects
 				(font
@@
 		)
 		(property "Datasheet" "~"
-			(at 69.85 109.22 0)
+			(at 69.85 105.41 0)
 			(effects
 				(font
@@
 		)
 		(property "Description" "Special symbol for telling ERC where power comes from"
-			(at 69.85 109.22 0)
+			(at 69.85 105.41 0)
 			(effects
 				(font

Commit message: lots of big updates
Parts:
- renumbered C26 to C31, C27 to C32, C28 to C33, C29 to C34, C30 to C35, C31 to C36, C32 to C37, C33 to C38, C34 to C39, C35 to C40, J9 to J10, J10 to J11, J15 to J9, R63 to R71, R64 to R72, R65 to R73, R66 to R74, R67 to R75, R68 to R76, U11 to U12, U12 to U13, U13 to U14

Commit message: first pass at ltc7004
Parts:
- removed J10, J11: Screw_Terminal_01x12, yarrboard:Busbar Rev D, symbol Connector:Screw_Terminal_01x12
- added J10, J11: Screw_Terminal_01x08, yarrboard:Busbar Rev D, symbol Connector:Screw_Terminal_01x08
- renumbered C31 to C52, C32 to C53, C33 to C54, C34 to C55, C35 to C56, C36 to C57, C37 to C58, C38 to C59, C39 to C60, C40 to C61, D29 to D45, D30 to D46, D31 to D47, D32 to D48, D33 to D49, R71 to R39, R72 to R40, R73 to R41, R74 to R42, R75 to R43, R76 to R44, U12 to U19, U13 to U20, U14 to U21
Connections:
- net +24V: now also J10.1 (Pin_1), J10.2 (Pin_2), J10.3 (Pin_3), J10.4 (Pin_4), J10.5 (Pin_5), J10.6 (Pin_6), J10.7 (Pin_7), J10.8 (Pin_8)
- net GNDA: now also J11.1 (Pin_1), J11.2 (Pin_2), J11.3 (Pin_3), J11.4 (Pin_4), J11.5 (Pin_5), J11.6 (Pin_6), J11.7 (Pin_7), J11.8 (Pin_8)
Other:
- title: FrothFET 12CH -> FrothFET 8CH
