File: frothfet-12ch/voltage_adc.kicad_sch (KiCad schematic)
At the start: 3 parts, among them U20 ADS1015IDGS

Commit message: schematic looking clean.
Parts:
- U20: LCSC (none) -> C193969; Mouser (none) -> 595-ADS1015IDGSR
Changed lines of the file:
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@@
+			)
+		)
+		(property "LCSC" "C193969"
+			(at 138.43 96.52 0)
+			(effects
+				(font
+					(size 1.27 1.27)
+				)
+				(hide yes)
+			)
+		)
+		(property "Mouser" " 595-ADS1015IDGSR "
+			(at 138.43 96.52 0)
+			(effects
+				(font
+					(size 1.27 1.27)
+				)
+				(hide yes)
 			)
 		)

Commit message: updated bom
Parts:
- C50: LCSC (none) -> C49678; Mouser 08053C104KAT4A -> (none)
- R110: LCSC (none) -> C84376
Changed lines of the file:
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@@
 			)
 		)
-		(property "Mouser" "08053C104KAT4A"
+		(property "Mouser" ""
+			(at 167.64 83.82 0)
+			(effects
+				(font
+					(size 1.27 1.27)
+				)
+				(hide yes)
+			)
+		)
+		(property "LCSC" "C49678"
 			(at 167.64 83.82 0)
 			(effects
@@
 			)
 		)
-		(property "LCSC" ""
-			(at 157.48 83.82 0)
-			(effects
+		(property "LCSC" "C84376"
+			(at 157.48 83.82 0)
+			(effects

Commit message: just need to route it...
Other:
- company: (none) -> https://github.com/hoeken/frothfet
- title: (none) -> FrothFET 12CH
Changed lines of the file:
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@@
 	(generator_version "8.0")
 	(paper "A4")
+	(title_block
+		(title "FrothFET 12CH")
+		(date "2024-08-17")
+		(rev "D")
+		(company "https://github.com/hoeken/frothfet")
+	)
 	(junction
 		(at 157.48 77.47)

Commit message: starting the mega route.
Parts:
- added C54: 10uF, Capacitor_SMD:C_0805_2012Metric_Pad1.18x1.45mm_HandSolder, symbol Device:C_Small
Connections:
- net +3.3V: now also C54.1
- net GNDA: now also C54.2
Other:
- moved on the sheet: C50
Changed lines of the file:
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@@
 		(color 0 0 0 0)
 	)
+	(junction
+		(at 167.64 77.47)
+		(diameter 0)
+		(color 0 0 0 0)
+	)
+	(junction
+		(at 167.64 107.95)
+		(diameter 0)
+		(color 0 0 0 0)
+	)
 	(wire
 		(pts
@@
 	(wire
 		(pts
+			(xy 180.34 93.98) (xy 180.34 107.95)
+		)
+		(stroke
+			(width 0)
+			(type default)
+		)
+	)
+	(wire
+		(pts
+			(xy 167.64 77.47) (xy 180.34 77.47)
+		)
+		(stroke
+			(width 0)
+			(type default)
+		)
+	)
+	(wire
+		(pts
 			(xy 123.19 99.06) (xy 128.27 99.06)
 		)
@@
 	(wire
 		(pts
+			(xy 180.34 77.47) (xy 180.34 88.9)
+		)
+		(stroke
+			(width 0)
+			(type default)
+		)
+	)
+	(wire
+		(pts
 			(xy 138.43 107.95) (xy 138.43 109.22)
 		)
@@
 	(wire
 		(pts
+			(xy 180.34 107.95) (xy 167.64 107.95)
+		)
+		(stroke
+			(width 0)
+			(type default)
+		)
+	)
+	(wire
+		(pts
 			(xy 148.59 91.44) (xy 157.48 91.44)
 		)
@@
 	(wire
 		(pts
-			(xy 167.64 86.36) (xy 167.64 107.95)
-		)
-		(stroke
-			(width 0)
-			(type default)
-		)
-	)
-	(wire
-		(pts
-			(xy 167.64 77.47) (xy 167.64 81.28)
+			(xy 167.64 93.98) (xy 167.64 107.95)
+		)
+		(stroke
+			(width 0)
+			(type default)
+		)
+	)
+	(wire
+		(pts
+			(xy 167.64 77.47) (xy 167.64 88.9)
 		)
 		(stroke
@@
 	(symbol
 		(lib_id "Device:C_Small")
-		(at 167.64 83.82 0)
+		(at 167.64 91.44 0)
 		(unit 1)
 		(exclude_from_sim no)
@@
 		(dnp no)
 		(property "Reference" "C50"
-			(at 170.18 82.5563 0)
+			(at 170.18 90.1763 0)
 			(effects
 				(font
@@
 		)
 		(property "Value" "100nF"
-			(at 170.18 85.0963 0)
+			(at 170.18 92.7163 0)
 			(effects
 				(font
@@
 		)
 		(property "Footprint" "Capacitor_SMD:C_0805_2012Metric_Pad1.18x1.45mm_HandSolder"
-			(at 167.64 83.82 0)
+			(at 167.64 91.44 0)
 			(effects
 				(font
@@
 		)
 		(property "Datasheet" "~"
-			(at 167.64 83.82 0)
+			(at 167.64 91.44 0)
 			(effects
 				(font
@@
 		)
 		(property "Description" ""
-			(at 167.64 83.82 0)
+			(at 167.64 91.44 0)
 			(effects
 				(font
@@
 		)
 		(property "Mouser" ""
-			(at 167.64 83.82 0)
+			(at 167.64 91.44 0)
 			(effects
 				(font
@@
 		)
 		(property "LCSC" "C49678"
-			(at 167.64 83.82 0)
+			(at 167.64 91.44 0)
 			(effects
 				(font
@@
 					(unit 1)
 				)
+			)
+		)
+	)
+	(symbol
+		(lib_id "Device:C_Small")
+		(at 180.34 91.44 0)
+		(unit 1)
+		(exclude_from_sim no)
+		(in_bom yes)
+		(on_board yes)
+		(dnp no)
+		(property "Reference" "C54"
+			(at 182.88 90.1763 0)
+			(effects
+				(font
+					(size 1.27 1.27)
+				)
+				(justify left)
+			)
+		)
+		(property "Value" "10uF"
+			(at 182.88 92.7163 0)
+			(effects
+				(font
+					(size 1.27 1.27)
+				)
+				(justify left)
+			)
+		)
+		(property "Footprint" "Capacitor_SMD:C_0805_2012Metric_Pad1.18x1.45mm_HandSolder"
+			(at 180.34 91.44 0)
+			(effects
+				(font
+					(size 1.27 1.27)
+				)
+				(hide yes)
+			)
+		)
+		(property "Datasheet" "~"
+			(at 180.34 91.44 0)
+			(effects
+				(font
+					(size 1.27 1.27)
+				)
+				(hide yes)
+			)
+		)
+		(property "Description" ""
+			(at 180.34 91.44 0)
+			(effects
+				(font
+					(size 1.27 1.27)
+				)
+				(hide yes)
+			)
+		)
+		(property "Vendor" ""
+			(at 180.34 91.44 0)
+			(effects
+				(font
+					(size 1.27 1.27)
+				)
+				(hide yes)
+			)
+		)
+		(property "LCSC" "C1952580"
+			(at 180.34 91.44 0)
+			(effects
+				(font
+					(size 1.27 1.27)
+				)
+				(hide yes)
+			)
+		)
+		(pin "1"
+		)
+		(pin "2"
+		)
+		(instances
+			(project "frothfet-12ch"
+				(path "/c83c6236-96e9-46ad-9d7a-9e2efa4a7966/a6260305-24e3-4714-b441-a7a157c17bd9"
+					(reference "C55")
+					(unit 1)
+				)
+				(path "/c83c6236-96e9-46ad-9d7a-9e2efa4a7966/bb9dea8b-8412-49bc-950d-dce57727bcd2"
+					(reference "C54")
+					(unit 1)
+				)
+				(path "/c83c6236-96e9-46ad-9d7a-9e2efa4a7966/efce81b0-0da6-4cc8-a856-27910d231a7d"
+					(reference "C56")
+					(unit 1)
+				)

Commit message: fully routed
Parts:
- renumbered C54 to C55
Changed lines of the file:
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@@
 		(on_board yes)
 		(dnp no)
-		(property "Reference" "C54"
+		(property "Reference" "C55"
 			(at 182.88 90.1763 0)
 			(effects

Commit message: lots of big updates
Parts:
- renumbered C50 to C58, C55 to C59, U20 to U21
Changed lines of the file:
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@@
 		(on_board yes)
 		(dnp no)
-		(property "Reference" "C50"
+		(property "Reference" "C58"
 			(at 170.18 90.1763 0)
 			(effects
@@
 			(project "8ch-mosfet"
 				(path "/c83c6236-96e9-46ad-9d7a-9e2efa4a7966/a6260305-24e3-4714-b441-a7a157c17bd9"
-					(reference "C50")
-					(unit 1)
-				)
-				(path "/c83c6236-96e9-46ad-9d7a-9e2efa4a7966/bb9dea8b-8412-49bc-950d-dce57727bcd2"
-					(reference "C49")
-					(unit 1)
-				)
-				(path "/c83c6236-96e9-46ad-9d7a-9e2efa4a7966/efce81b0-0da6-4cc8-a856-27910d231a7d"
-					(reference "C51")
+					(reference "C58")
+					(unit 1)
+				)
+				(path "/c83c6236-96e9-46ad-9d7a-9e2efa4a7966/bb9dea8b-8412-49bc-950d-dce57727bcd2"
+					(reference "C56")
 					(unit 1)
 				)
@@
 		(dnp no)
 		(fields_autoplaced yes)
-		(property "Reference" "U20"
+		(property "Reference" "U21"
 			(at 140.6241 81.28 0)
 			(effects
@@
 			(project "8ch-mosfet"
 				(path "/c83c6236-96e9-46ad-9d7a-9e2efa4a7966/a6260305-24e3-4714-b441-a7a157c17bd9"
+					(reference "U21")
+					(unit 1)
+				)
+				(path "/c83c6236-96e9-46ad-9d7a-9e2efa4a7966/bb9dea8b-8412-49bc-950d-dce57727bcd2"
 					(reference "U20")
-					(unit 1)
-				)
-				(path "/c83c6236-96e9-46ad-9d7a-9e2efa4a7966/bb9dea8b-8412-49bc-950d-dce57727bcd2"
-					(reference "U19")
-					(unit 1)
-				)
-				(path "/c83c6236-96e9-46ad-9d7a-9e2efa4a7966/efce81b0-0da6-4cc8-a856-27910d231a7d"
-					(reference "U21")
 					(unit 1)
 				)
@@
 		(on_board yes)
 		(dnp no)
-		(property "Reference" "C55"
+		(property "Reference" "C59"
 			(at 182.88 90.1763 0)
 			(effects
@@
 			(project "frothfet-12ch"
 				(path "/c83c6236-96e9-46ad-9d7a-9e2efa4a7966/a6260305-24e3-4714-b441-a7a157c17bd9"
-					(reference "C55")
-					(unit 1)
-				)
-				(path "/c83c6236-96e9-46ad-9d7a-9e2efa4a7966/bb9dea8b-8412-49bc-950d-dce57727bcd2"
-					(reference "C54")
-					(unit 1)
-				)
-				(path "/c83c6236-96e9-46ad-9d7a-9e2efa4a7966/efce81b0-0da6-4cc8-a856-27910d231a7d"
-					(reference "C56")
+					(reference "C59")
+					(unit 1)
+				)
+				(path "/c83c6236-96e9-46ad-9d7a-9e2efa4a7966/bb9dea8b-8412-49bc-950d-dce57727bcd2"
+					(reference "C57")
 					(unit 1)
 				)
@@
 					(unit 1)
 				)
-				(path "/c83c6236-96e9-46ad-9d7a-9e2efa4a7966/efce81b0-0da6-4cc8-a856-27910d231a7d"
-					(reference "R111")
-					(unit 1)
-				)
 			)
 		)
@@
 		(on_board yes)
 		(dnp no)
-		(property "Reference" "#PWR0107"
+		(property "Reference" "#PWR0122"
 			(at 138.43 115.57 0)
 			(effects
@@
 			(project "8ch-mosfet"
 				(path "/c83c6236-96e9-46ad-9d7a-9e2efa4a7966/a6260305-24e3-4714-b441-a7a157c17bd9"
-					(reference "#PWR0107")
-					(unit 1)
-				)
-				(path "/c83c6236-96e9-46ad-9d7a-9e2efa4a7966/bb9dea8b-8412-49bc-950d-dce57727bcd2"
-					(reference "#PWR0105")
-					(unit 1)
-				)
-				(path "/c83c6236-96e9-46ad-9d7a-9e2efa4a7966/efce81b0-0da6-4cc8-a856-27910d231a7d"
-					(reference "#PWR0109")
+					(reference "#PWR0122")
+					(unit 1)
+				)
+				(path "/c83c6236-96e9-46ad-9d7a-9e2efa4a7966/bb9dea8b-8412-49bc-950d-dce57727bcd2"
+					(reference "#PWR0120")
 					(unit 1)
 				)
@@
 		(dnp no)
 		(fields_autoplaced yes)
-		(property "Reference" "#PWR0106"
+		(property "Reference" "#PWR0121"
 			(at 138.43 80.01 0)
 			(effects
@@
 			(project "8ch-mosfet"
 				(path "/c83c6236-96e9-46ad-9d7a-9e2efa4a7966/a6260305-24e3-4714-b441-a7a157c17bd9"
-					(reference "#PWR0106")
-					(unit 1)
-				)
-				(path "/c83c6236-96e9-46ad-9d7a-9e2efa4a7966/bb9dea8b-8412-49bc-950d-dce57727bcd2"
-					(reference "#PWR0104")
-					(unit 1)
-				)
-				(path "/c83c6236-96e9-46ad-9d7a-9e2efa4a7966/efce81b0-0da6-4cc8-a856-27910d231a7d"
-					(reference "#PWR0108")
-					(unit 1)
-				)
+					(reference "#PWR0121")
+					(unit 1)
+				)
+				(path "/c83c6236-96e9-46ad-9d7a-9e2efa4a7966/bb9dea8b-8412-49bc-950d-dce57727bcd2"
+					(reference "#PWR0119")
+					(unit 1)
+				)

Commit message: first pass at ltc7004
Parts:
- renumbered C58 to C64, C59 to C65, R110 to R46, U21 to U23
Other:
- title: FrothFET 12CH -> FrothFET 8CH
Changed lines of the file:
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@@
 	(paper "A4")
 	(title_block
-		(title "FrothFET 12CH")
-		(date "2024-08-17")
+		(title "FrothFET 8CH")
+		(date "2024-08-21")
 		(rev "D")
 		(company "https://github.com/hoeken/frothfet")
@@
 		(on_board yes)
 		(dnp no)
-		(property "Reference" "C58"
+		(property "Reference" "C64"
 			(at 170.18 90.1763 0)
 			(effects
@@
 			(project "8ch-mosfet"
 				(path "/c83c6236-96e9-46ad-9d7a-9e2efa4a7966/a6260305-24e3-4714-b441-a7a157c17bd9"
-					(reference "C58")
+					(reference "C64")
 					(unit 1)
 				)
 				(path "/c83c6236-96e9-46ad-9d7a-9e2efa4a7966/bb9dea8b-8412-49bc-950d-dce57727bcd2"
-					(reference "C56")
+					(reference "C62")
 					(unit 1)
 				)
@@
 		(dnp no)
 		(fields_autoplaced yes)
-		(property "Reference" "U21"
+		(property "Reference" "U23"
 			(at 140.6241 81.28 0)
 			(effects
@@
 			(project "8ch-mosfet"
 				(path "/c83c6236-96e9-46ad-9d7a-9e2efa4a7966/a6260305-24e3-4714-b441-a7a157c17bd9"
-					(reference "U21")
+					(reference "U23")
 					(unit 1)
 				)
 				(path "/c83c6236-96e9-46ad-9d7a-9e2efa4a7966/bb9dea8b-8412-49bc-950d-dce57727bcd2"
-					(reference "U20")
+					(reference "U22")
 					(unit 1)
 				)
@@
 		(on_board yes)
 		(dnp no)
-		(property "Reference" "C59"
+		(property "Reference" "C65"
 			(at 182.88 90.1763 0)
 			(effects
@@
 			(project "frothfet-12ch"
 				(path "/c83c6236-96e9-46ad-9d7a-9e2efa4a7966/a6260305-24e3-4714-b441-a7a157c17bd9"
-					(reference "C59")
+					(reference "C65")
 					(unit 1)
 				)
 				(path "/c83c6236-96e9-46ad-9d7a-9e2efa4a7966/bb9dea8b-8412-49bc-950d-dce57727bcd2"
-					(reference "C57")
+					(reference "C63")
 					(unit 1)
 				)
@@
 		(dnp no)
 		(fields_autoplaced yes)
-		(property "Reference" "R110"
+		(property "Reference" "R46"
 			(at 160.02 82.55 0)
 			(effects
@@
 			(project "8ch-mosfet"
 				(path "/c83c6236-96e9-46ad-9d7a-9e2efa4a7966/a6260305-24e3-4714-b441-a7a157c17bd9"
-					(reference "R110")
+					(reference "R46")
 					(unit 1)
 				)
 				(path "/c83c6236-96e9-46ad-9d7a-9e2efa4a7966/bb9dea8b-8412-49bc-950d-dce57727bcd2"
-					(reference "R109")
+					(reference "R45")
 					(unit 1)
 				)
@@
 		(on_board yes)
 		(dnp no)
-		(property "Reference" "#PWR0122"
+		(property "Reference" "#PWR072"
 			(at 138.43 115.57 0)
 			(effects
@@
 			(project "8ch-mosfet"
 				(path "/c83c6236-96e9-46ad-9d7a-9e2efa4a7966/a6260305-24e3-4714-b441-a7a157c17bd9"
-					(reference "#PWR0122")
+					(reference "#PWR072")
 					(unit 1)
 				)
 				(path "/c83c6236-96e9-46ad-9d7a-9e2efa4a7966/bb9dea8b-8412-49bc-950d-dce57727bcd2"
-					(reference "#PWR0120")
+					(reference "#PWR070")
 					(unit 1)
 				)
@@
 		(dnp no)
 		(fields_autoplaced yes)
-		(property "Reference" "#PWR0121"
+		(property "Reference" "#PWR071"
 			(at 138.43 80.01 0)
 			(effects
@@
 			(project "8ch-mosfet"
 				(path "/c83c6236-96e9-46ad-9d7a-9e2efa4a7966/a6260305-24e3-4714-b441-a7a157c17bd9"
-					(reference "#PWR0121")
+					(reference "#PWR071")
 					(unit 1)
 				)
 				(path "/c83c6236-96e9-46ad-9d7a-9e2efa4a7966/bb9dea8b-8412-49bc-950d-dce57727bcd2"
-					(reference "#PWR0119")
-					(unit 1)
-				)
+					(reference "#PWR069")
+					(unit 1)
+				)
