File: revisions/FrothFET-Rev-D/FrothFET-Rev-D.kicad_pcb (KiCad board)
At the start: 4 copper layers, 144 x 127 mm, 252 parts, among them J1 Conn_01x01, J10 Screw_Terminal_01x08, J11 Screw_Terminal_01x08, J12 Conn_01x03_Pin, J2 Conn_01x01, J3 Conn_01x01, J4 Conn_01x01, J5 Conn_01x01, J6 Conn_01x01, J7 Conn_01x01, J8 Conn_01x01, J9 Conn_01x03_Pin, Q1 BSC010N04LS, Q10 2N7002, Q2 BSC010N04LS, Q3 BSC010N04LS, Q4 BSC010N04LS, Q5 BSC010N04LS, Q6 BSC010N04LS, Q7 BSC010N04LS, Q8 BSC010N04LS, Q9 2N7002, U1 ESP32-S3-DEVKITC, U10 LTC7004EMSE-PBF, U11 ACS725xLCTR-20AU, U12 LTC7004EMSE-PBF, U13 ACS725xLCTR-20AU, U14 LTC7004EMSE-PBF, U15 ACS725xLCTR-20AU, U16 LTC7004EMSE-PBF, U17 ACS725xLCTR-20AU, U18 MCP3564R, U19 MCP1502-33, U2 LTC7004EMSE-PBF, U20 MCP3425A0T-ECH, U21 XL1509-5.0, U22 ADS1015IDGS, U23 ADS1015IDGS, U24 MCP1754S-3302xCB, U3 ACS725xLCTR-20AU, U4 LTC7004EMSE-PBF, U5 ACS725xLCTR-20AU, U6 LTC7004EMSE-PBF, U7 ACS725xLCTR-20AU, U8 LTC7004EMSE-PBF, U9 ACS725xLCTR-20AU

Commit message: tweaks to rev d
Parts:
- C15, C21, C27, C3, C33, C39, C45, C9: value 100nF -> 220nF
- R10, R16, R22, R28, R34, R4, R40, R46: value 300K 0.1% -> 4.7K 0.1%
- R11, R17, R23, R29, R35, R41, R47, R5: value 22K 0.1% -> 560 0.1%
- R12, R18, R24, R30, R36, R42, R48, R6: value 0R -> 10R
- R63, R64, R65, R66, R67, R68, R69, R70: value 0R -> 150K
Connections:
- U1 pad 20: unconnected-(U1-GPIO14-Pad20) -> /HIRES ADC1/IRQ
- U18 pad 17: unconnected-(U18-~{IRQ}-Pad17) -> /HIRES ADC1/IRQ
