File: revisions/FrothFET-Rev-D/power.kicad_sch (KiCad schematic)
At the start: 36 parts, among them J10 Screw_Terminal_01x08, J11 Screw_Terminal_01x08, J12 Conn_01x03_Pin, J9 Conn_01x03_Pin, U19 MCP1502-33, U20 MCP3425A0T-ECH, U21 XL1509-5.0, U24 MCP1754S-3302xCB

Commit message: tweaks to rev d
Parts:
- C74, U19, U24: now left out of the parts list
Changed lines of the file:
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@@
 		(unit 1)
 		(exclude_from_sim no)
-		(in_bom yes)
+		(in_bom no)
 		(on_board yes)
 		(dnp yes)
@@
 		(unit 1)
 		(exclude_from_sim no)
-		(in_bom yes)
+		(in_bom no)
 		(on_board yes)
 		(dnp yes)
@@
 		(unit 1)
 		(exclude_from_sim no)
-		(in_bom yes)
+		(in_bom no)
 		(on_board yes)
 		(dnp yes)
