File: frothfet/frothfet.kicad_sch (KiCad schematic)
At the start: 11 parts, among them U1 74AHC541

Commit message: added test points
Parts:
- added TP1, TP2: ~, TestPoint:TestPoint_THTPad_D1.5mm_Drill0.7mm, symbol Connector:TestPoint
Connections:
- net SCL: now also TP2.1
- net SDA: now also TP1.1
Changed lines of the file:
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@@
 	)
 	(junction
+		(at 81.28 110.49)
+		(diameter 0)
+		(color 0 0 0 0)
+	)
+	(junction
+		(at 81.28 107.95)
+		(diameter 0)
+		(color 0 0 0 0)
+	)
+	(junction
 		(at 60.96 31.75)
 		(diameter 0)
@@
 	(wire
 		(pts
+			(xy 81.28 110.49) (xy 107.95 110.49)
+		)
+		(stroke
+			(width 0)
+			(type default)
+		)
+	)
+	(wire
+		(pts
 			(xy 107.95 71.12) (xy 73.66 71.12)
 		)
@@
 	(wire
 		(pts
+			(xy 81.28 107.95) (xy 107.95 107.95)
+		)
+		(stroke
+			(width 0)
+			(type default)
+		)
+	)
+	(wire
+		(pts
 			(xy 73.66 63.5) (xy 73.66 66.04)
 		)
@@
 	(wire
 		(pts
-			(xy 69.85 107.95) (xy 107.95 107.95)
+			(xy 69.85 107.95) (xy 81.28 107.95)
 		)
 		(stroke
@@
 	(wire
 		(pts
-			(xy 59.69 110.49) (xy 107.95 110.49)
+			(xy 59.69 110.49) (xy 81.28 110.49)
 		)
 		(stroke
@@
 	)
 	(symbol
+		(lib_id "Connector:TestPoint")
+		(at 81.28 110.49 180)
+		(unit 1)
+		(exclude_from_sim no)
+		(in_bom no)
+		(on_board yes)
+		(dnp no)
+		(property "Reference" "TP2"
+			(at 82.804 115.57 0)
+			(effects
+				(font
+					(size 1.27 1.27)
+				)
+				(justify left)
+			)
+		)
+		(property "Value" "~"
+			(at 78.74 112.5221 0)
+			(effects
+				(font
+					(size 1.27 1.27)
+				)
+				(justify left)
+				(hide yes)
+			)
+		)
+		(property "Footprint" "TestPoint:TestPoint_THTPad_D1.5mm_Drill0.7mm"
+			(at 76.2 110.49 0)
+			(effects
+				(font
+					(size 1.27 1.27)
+				)
+				(hide yes)
+			)
+		)
+		(property "Datasheet" "~"
+			(at 76.2 110.49 0)
+			(effects
+				(font
+					(size 1.27 1.27)
+				)
+				(hide yes)
+			)
+		)
+		(property "Description" "test point"
+			(at 81.28 110.49 0)
+			(effects
+				(font
+					(size 1.27 1.27)
+				)
+				(hide yes)
+			)
+		)
+		(pin "1"
+		)
+		(instances
+			(project "frothfet"
+				(path "/c83c6236-96e9-46ad-9d7a-9e2efa4a7966"
+					(reference "TP2")
+					(unit 1)
+				)
+			)
+		)
+	)
+	(symbol
 		(lib_id "power:+3.3V")
 		(at 215.9 113.03 270)
@@
 	)
 	(symbol
+		(lib_id "Connector:TestPoint")
+		(at 81.28 107.95 0)
+		(unit 1)
+		(exclude_from_sim no)
+		(in_bom no)
+		(on_board yes)
+		(dnp no)
+		(property "Reference" "TP1"
+			(at 79.756 102.87 0)
+			(effects
+				(font
+					(size 1.27 1.27)
+				)
+				(justify left)
+			)
+		)
+		(property "Value" "~"
+			(at 83.82 105.9179 0)
+			(effects
+				(font
+					(size 1.27 1.27)
+				)
+				(justify left)
+				(hide yes)
+			)
+		)
+		(property "Footprint" "TestPoint:TestPoint_THTPad_D1.5mm_Drill0.7mm"
+			(at 86.36 107.95 0)
+			(effects
+				(font
+					(size 1.27 1.27)
+				)
+				(hide yes)
+			)
+		)
+		(property "Datasheet" "~"
+			(at 86.36 107.95 0)
+			(effects
+				(font
+					(size 1.27 1.27)
+				)
+				(hide yes)
+			)
+		)
+		(property "Description" "test point"
+			(at 81.28 107.95 0)
+			(effects
+				(font
+					(size 1.27 1.27)
+				)
+				(hide yes)
+			)
+		)
+		(pin "1"
+		)
+		(instances
+			(project "frothfet"
+				(path "/c83c6236-96e9-46ad-9d7a-9e2efa4a7966"
+					(reference "TP1")
+					(unit 1)
+				)
+			)
+		)
+	)
+	(symbol
 		(lib_id "power:GND")
 		(at 215.9 71.12 90)
@@
 		(on_board yes)
 		(dnp no)
-		(property "Reference" "#PWR1"
+		(property "Reference" "#PWR01"
 			(at 43.18 180.34 0)
 			(effects
@@
 			(project "8ch-mosfet"
 				(path "/c83c6236-96e9-46ad-9d7a-9e2efa4a7966"
-					(reference "#PWR1")
+					(reference "#PWR01")
 					(unit 1)
 				)

Commit message: worked on routing load channel.
Parts:
- added J1: Conn_01x10, Connector_PinHeader_2.54mm:PinHeader_1x10_P2.54mm_Vertical, symbol Connector_Generic:Conn_01x10
- added J2: Conn_01x04_MountingPin, yarrboard:JST_SH_BM04B-SRSS-TB_1x04-1MP_P1.00mm_Vertical, symbol Connector_Generic_MountingPin:Conn_01x04_MountingPin
- H1, H2, H3, H4: footprint MountingHole:MountingHole_3.2mm_M3_DIN965_Pad -> yarrboard:SMTSO30XXX
Connections:
- net +3.3V: now also J1.1 (Pin_1), J2.2 (Pin_2)
- net GND: now also J1.10 (Pin_10), J2.1 (Pin_1), J2.MP (MountPin)
- net SCL: now also J2.4 (Pin_4)
- net SDA: now also J2.3 (Pin_3)
- new net GPIO15: J1.2 (Pin_2)
- new net GPIO16: J1.3 (Pin_3)
- new net GPIO17: J1.4 (Pin_4)
- new net GPIO18: J1.5 (Pin_5)
- new net GPIO39: J1.6 (Pin_6)
- new net GPIO40: J1.7 (Pin_7)
- new net GPIO41: J1.8 (Pin_8)
- new net GPIO42: J1.9 (Pin_9)
- no-connect marks 22 -> 14
Other:
- note added: "ACCESSORIES"
- note added: "ESP32-S3"
- note added: "I2C / QWIIC"
- note added: "LOAD DRIVERS - 8 CHANNELS"
- note added: "MOUNTING HOLES"
- note added: "POWER SUPPLY"
- note removed: "ESP32-S3 Module"
- moved on the sheet: H1, H2, H3, H4, LOADS1, R1, R2
