File: frothfet/esp32-s3.kicad_sch (KiCad schematic)
At the start: 28 parts, among them J3 USB_TYPE_C_16PIN, J4 Conn_01x04, SW1 BOOT, SW2 RESET, U28 ESP32-S3-WROOM-1-N16R8, U29 USBLC6-2SC6, U30 SN74LV1T34DBV, U31 XC6210B332MR

Commit message: added the buffer circuit
Parts:
- renumbered C62 to C63, C63 to C64, C64 to C65, C65 to C66, C66 to C67, C67 to C68, C68 to C69, C69 to C70, C70 to C71, C71 to C72, R50 to R59, R51 to R60, R52 to R61, R53 to R62, U28 to U29, U29 to U30, U30 to U31, U31 to U32

Commit message: added test points
Parts:
- added D37: GREEN, LED_SMD:LED_0603_1608Metric, symbol Device:LED
- added R54: 5.1k, Resistor_SMD:R_0603_1608Metric, symbol Device:R_Small_US
- renumbered C63 to C62, C64 to C63, C65 to C64, C66 to C65, C67 to C66, C68 to C67, C70 to C68, C72 to C70, D36 to D35, D37 to D36, FB3 to FB2, R59 to R50, R60 to R51, R61 to R52, R62 to R53, TP2 to TP26, TP4 to TP27, TP3 to TP28, U29 to U30, U30 to U31, U31 to U32, U32 to U33
Connections:
- net +3.3V: now also D37.2 (A)
- net GND: now also R54.2
- new net: D37.1 (K), R54.1
Other:
- moved on the sheet: C68, C70, TP27, U33

Commit message: worked on routing load channel.
Parts:
- renumbered J3 to J12, J4 to J13, TP26 to TP25, TP27 to TP26, TP28 to TP27
Other:
- company: (none) -> https://github.com/hoeken/frothfet
- title: https://github.com/hoeken/brineomatic -> FrothFET 8CH
Changed lines of the file:
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@@
 	(paper "A4")
 	(title_block
-		(title "https://github.com/hoeken/brineomatic")
-		(date "2025-08-28")
-		(rev "C")
+		(title "FrothFET 8CH")
+		(date "2024-08-21")
+		(rev "F")
+		(company "https://github.com/hoeken/frothfet")
 	)
 	(rectangle
@@
 		(on_board yes)
 		(dnp no)
-		(property "Reference" "#PWR0136"
+		(property "Reference" "#PWR0141"
 			(at 97.79 179.07 0)
 			(effects
@@
 			(project "frothfet"
 				(path "/c83c6236-96e9-46ad-9d7a-9e2efa4a7966/777fe0ac-daa5-4cfe-9bd1-5eba0a425019"
-					(reference "#PWR0136")
+					(reference "#PWR0141")
 					(unit 1)
 				)
@@
 		(on_board yes)
 		(dnp no)
-		(property "Reference" "#PWR0148"
+		(property "Reference" "#PWR0153"
 			(at 220.98 119.38 0)
 			(effects
@@
 			(project "frothfet"
 				(path "/c83c6236-96e9-46ad-9d7a-9e2efa4a7966/777fe0ac-daa5-4cfe-9bd1-5eba0a425019"
-					(reference "#PWR0148")
+					(reference "#PWR0153")
 					(unit 1)
 				)
@@
 		(dnp no)
 		(fields_autoplaced yes)
-		(property "Reference" "#PWR0140"
+		(property "Reference" "#PWR0145"
 			(at 115.57 81.28 0)
 			(effects
@@
 			(project "frothfet"
 				(path "/c83c6236-96e9-46ad-9d7a-9e2efa4a7966/777fe0ac-daa5-4cfe-9bd1-5eba0a425019"
-					(reference "#PWR0140")
+					(reference "#PWR0145")
 					(unit 1)
 				)
@@
 		(on_board yes)
 		(dnp no)
-		(property "Reference" "#PWR0142"
+		(property "Reference" "#PWR0147"
 			(at 163.83 31.75 0)
 			(effects
@@
 			(project "frothfet"
 				(path "/c83c6236-96e9-46ad-9d7a-9e2efa4a7966/777fe0ac-daa5-4cfe-9bd1-5eba0a425019"
-					(reference "#PWR0142")
+					(reference "#PWR0147")
 					(unit 1)
 				)
@@
 		(dnp no)
 		(fields_autoplaced yes)
-		(property "Reference" "#FLG09"
+		(property "Reference" "#FLG010"
 			(at 125.73 37.465 0)
 			(effects
@@
 			(project "frothfet"
 				(path "/c83c6236-96e9-46ad-9d7a-9e2efa4a7966/777fe0ac-daa5-4cfe-9bd1-5eba0a425019"
-					(reference "#FLG09")
+					(reference "#FLG010")
 					(unit 1)
 				)
@@
 		(on_board yes)
 		(dnp no)
-		(property "Reference" "#PWR0147"
+		(property "Reference" "#PWR0152"
 			(at 213.36 64.77 0)
 			(effects
@@
 			(project "frothfet"
 				(path "/c83c6236-96e9-46ad-9d7a-9e2efa4a7966/777fe0ac-daa5-4cfe-9bd1-5eba0a425019"
-					(reference "#PWR0147")
+					(reference "#PWR0152")
 					(unit 1)
 				)
@@
 		(dnp yes)
 		(fields_autoplaced yes)
-		(property "Reference" "J4"
+		(property "Reference" "J13"
 			(at 121.92 179.0699 0)
 			(effects
@@
 			(project "frothfet"
 				(path "/c83c6236-96e9-46ad-9d7a-9e2efa4a7966/777fe0ac-daa5-4cfe-9bd1-5eba0a425019"
-					(reference "J4")
+					(reference "J13")
 					(unit 1)
 				)
@@
 		(on_board yes)
 		(dnp no)
-		(property "Reference" "#PWR0143"
+		(property "Reference" "#PWR0148"
 			(at 184.15 119.38 0)
 			(effects
@@
 			(project "frothfet"
 				(path "/c83c6236-96e9-46ad-9d7a-9e2efa4a7966/777fe0ac-daa5-4cfe-9bd1-5eba0a425019"
-					(reference "#PWR0143")
+					(reference "#PWR0148")
 					(unit 1)
 				)
@@
 		(on_board yes)
 		(dnp no)
-		(property "Reference" "TP27"
+		(property "Reference" "TP26"
 			(at 213.106 24.13 0)
 			(effects
@@
 			(project "frothfet"
 				(path "/c83c6236-96e9-46ad-9d7a-9e2efa4a7966/777fe0ac-daa5-4cfe-9bd1-5eba0a425019"
-					(reference "TP27")
+					(reference "TP26")
 					(unit 1)
 				)
@@
 		(dnp no)
 		(fields_autoplaced yes)
-		(property "Reference" "#PWR0137"
+		(property "Reference" "#PWR0142"
 			(at 97.79 186.69 0)
 			(effects
@@
 			(project "frothfet"
 				(path "/c83c6236-96e9-46ad-9d7a-9e2efa4a7966/777fe0ac-daa5-4cfe-9bd1-5eba0a425019"
-					(reference "#PWR0137")
+					(reference "#PWR0142")
 					(unit 1)
 				)
@@
 		(on_board yes)
 		(dnp no)
-		(property "Reference" "TP28"
+		(property "Reference" "TP27"
 			(at 214.376 118.11 0)
 			(effects
@@
 			(project "frothfet"
 				(path "/c83c6236-96e9-46ad-9d7a-9e2efa4a7966/777fe0ac-daa5-4cfe-9bd1-5eba0a425019"
-					(reference "TP28")
+					(reference "TP27")
 					(unit 1)
 				)
@@
 		(dnp no)
 		(fields_autoplaced yes)
-		(property "Reference" "#PWR0135"
+		(property "Reference" "#PWR0140"
 			(at 85.09 162.56 0)
 			(effects
@@
 			(project "frothfet"
 				(path "/c83c6236-96e9-46ad-9d7a-9e2efa4a7966/777fe0ac-daa5-4cfe-9bd1-5eba0a425019"
-					(reference "#PWR0135")
+					(reference "#PWR0140")
 					(unit 1)
 				)
@@
 		(dnp no)
 		(fields_autoplaced yes)
-		(property "Reference" "#PWR0146"
+		(property "Reference" "#PWR0151"
 			(at 204.47 83.82 0)
 			(effects
@@
 			(project "frothfet"
 				(path "/c83c6236-96e9-46ad-9d7a-9e2efa4a7966/777fe0ac-daa5-4cfe-9bd1-5eba0a425019"
-					(reference "#PWR0146")
+					(reference "#PWR0151")
 					(unit 1)
 				)
@@
 		(dnp no)
 		(fields_autoplaced yes)
-		(property "Reference" "#PWR0150"
+		(property "Reference" "#PWR0155"
 			(at 229.87 144.78 0)
 			(effects
@@
 			(project "frothfet"
 				(path "/c83c6236-96e9-46ad-9d7a-9e2efa4a7966/777fe0ac-daa5-4cfe-9bd1-5eba0a425019"
-					(reference "#PWR0150")
+					(reference "#PWR0155")
 					(unit 1)
 				)
@@
 		(dnp no)
 		(fields_autoplaced yes)
-		(property "Reference" "#PWR0144"
+		(property "Reference" "#PWR0149"
 			(at 193.04 143.51 0)
 			(effects
@@
 			(project "frothfet"
 				(path "/c83c6236-96e9-46ad-9d7a-9e2efa4a7966/777fe0ac-daa5-4cfe-9bd1-5eba0a425019"
-					(reference "#PWR0144")
+					(reference "#PWR0149")
 					(unit 1)
 				)
@@
 		(on_board yes)
 		(dnp no)
-		(property "Reference" "TP26"
+		(property "Reference" "TP25"
 			(at 177.546 118.11 0)
 			(effects
@@
 			(project "frothfet"
 				(path "/c83c6236-96e9-46ad-9d7a-9e2efa4a7966/777fe0ac-daa5-4cfe-9bd1-5eba0a425019"
-					(reference "TP26")
+					(reference "TP25")
 					(unit 1)
 				)
@@
 		(dnp no)
 		(fields_autoplaced yes)
-		(property "Reference" "#PWR0139"
+		(property "Reference" "#PWR0144"
 			(at 109.22 48.26 0)
 			(effects
@@
 			(project "frothfet"
 				(path "/c83c6236-96e9-46ad-9d7a-9e2efa4a7966/777fe0ac-daa5-4cfe-9bd1-5eba0a425019"
-					(reference "#PWR0139")
+					(reference "#PWR0144")
 					(unit 1)
 				)
@@
 		(on_board yes)
 		(dnp no)
-		(property "Reference" "#PWR0138"
+		(property "Reference" "#PWR0143"
 			(at 106.68 100.33 0)
 			(effects
@@
 			(project "frothfet"
 				(path "/c83c6236-96e9-46ad-9d7a-9e2efa4a7966/777fe0ac-daa5-4cfe-9bd1-5eba0a425019"
-					(reference "#PWR0138")
+					(reference "#PWR0143")
 					(unit 1)
 				)
@@
 		(dnp no)
 		(fields_autoplaced yes)
-		(property "Reference" "J3"
+		(property "Reference" "J12"
 			(at 68.58 27.94 0)
 			(effects
@@
 			(project "frothfet"
 				(path "/c83c6236-96e9-46ad-9d7a-9e2efa4a7966/777fe0ac-daa5-4cfe-9bd1-5eba0a425019"
-					(reference "J3")
+					(reference "J12")
 					(unit 1)
 				)
@@
 		(on_board yes)
 		(dnp no)
-		(property "Reference" "#PWR0149"
+		(property "Reference" "#PWR0154"
 			(at 224.79 31.75 0)
 			(effects
@@
 			(project "frothfet"
 				(path "/c83c6236-96e9-46ad-9d7a-9e2efa4a7966/777fe0ac-daa5-4cfe-9bd1-5eba0a425019"
-					(reference "#PWR0149")
+					(reference "#PWR0154")
 					(unit 1)
 				)
@@
 		(dnp no)
 		(fields_autoplaced yes)
-		(property "Reference" "#FLG08"
+		(property "Reference" "#FLG09"
 			(at 91.44 31.115 0)
 			(effects
@@
 			(project "frothfet"
 				(path "/c83c6236-96e9-46ad-9d7a-9e2efa4a7966/777fe0ac-daa5-4cfe-9bd1-5eba0a425019"
-					(reference "#FLG08")
+					(reference "#FLG09")
 					(unit 1)
 				)
@@
 		(dnp no)
 		(fields_autoplaced yes)
-		(property "Reference" "#PWR0134"
+		(property "Reference" "#PWR0139"
 			(at 64.77 80.01 0)
 			(effects
@@
 			(project "frothfet"
 				(path "/c83c6236-96e9-46ad-9d7a-9e2efa4a7966/777fe0ac-daa5-4cfe-9bd1-5eba0a425019"
-					(reference "#PWR0134")
+					(reference "#PWR0139")
 					(unit 1)
 				)
@@
 		(on_board yes)
 		(dnp no)
-		(property "Reference" "#PWR0141"
+		(property "Reference" "#PWR0146"
 			(at 125.73 36.83 0)
 			(effects
@@
 			(project "frothfet"
 				(path "/c83c6236-96e9-46ad-9d7a-9e2efa4a7966/777fe0ac-daa5-4cfe-9bd1-5eba0a425019"
-					(reference "#PWR0141")
+					(reference "#PWR0146")
 					(unit 1)
 				)
@@
 		(dnp no)
 		(fields_autoplaced yes)
-		(property "Reference" "#PWR0145"
+		(property "Reference" "#PWR0150"
 			(at 198.12 48.26 0)
 			(effects
@@
 			(project "frothfet"
 				(path "/c83c6236-96e9-46ad-9d7a-9e2efa4a7966/777fe0ac-daa5-4cfe-9bd1-5eba0a425019"
-					(reference "#PWR0145")
+					(reference "#PWR0150")
 					(unit 1)
 				)

Commit message: channel routing is basically done
Parts:
- renumbered R50 to R52, R51 to R53, R52 to R54, R53 to R55, R54 to R56
Changed lines of the file:
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@@
 		(on_board yes)
 		(dnp no)
-		(property "Reference" "R51"
+		(property "Reference" "R53"
 			(at 96.52 45.72 90)
 			(effects
@@
 			(project "frothfet"
 				(path "/c83c6236-96e9-46ad-9d7a-9e2efa4a7966/777fe0ac-daa5-4cfe-9bd1-5eba0a425019"
-					(reference "R51")
+					(reference "R53")
 					(unit 1)
 				)
@@
 		(dnp no)
 		(fields_autoplaced yes)
-		(property "Reference" "R54"
+		(property "Reference" "R56"
 			(at 237.49 38.0999 0)
 			(effects
@@
 			(project "frothfet"
 				(path "/c83c6236-96e9-46ad-9d7a-9e2efa4a7966/777fe0ac-daa5-4cfe-9bd1-5eba0a425019"
-					(reference "R54")
+					(reference "R56")
 					(unit 1)
 				)
@@
 		(dnp no)
 		(fields_autoplaced yes)
-		(property "Reference" "R52"
+		(property "Reference" "R54"
 			(at 186.69 118.1099 0)
 			(effects
@@
 			(project "frothfet"
 				(path "/c83c6236-96e9-46ad-9d7a-9e2efa4a7966/777fe0ac-daa5-4cfe-9bd1-5eba0a425019"
-					(reference "R52")
+					(reference "R54")
 					(unit 1)
 				)
@@
 		(on_board yes)
 		(dnp no)
-		(property "Reference" "R50"
+		(property "Reference" "R52"
 			(at 96.52 38.1 90)
 			(effects
@@
 			(project "frothfet"
 				(path "/c83c6236-96e9-46ad-9d7a-9e2efa4a7966/777fe0ac-daa5-4cfe-9bd1-5eba0a425019"
-					(reference "R50")
+					(reference "R52")
 					(unit 1)
 				)
@@
 		(dnp no)
 		(fields_autoplaced yes)
-		(property "Reference" "R53"
+		(property "Reference" "R55"
 			(at 223.52 118.1099 0)
 			(effects
@@
 			(project "frothfet"
 				(path "/c83c6236-96e9-46ad-9d7a-9e2efa4a7966/777fe0ac-daa5-4cfe-9bd1-5eba0a425019"
-					(reference "R53")
+					(reference "R55")
 					(unit 1)
 				)

Commit message: starting to layout the rest of the components.
Parts:
- renumbered J12 to J13, J13 to J14
Changed lines of the file:
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@@
 		(on_board yes)
 		(dnp no)
-		(property "Reference" "#PWR0141"
+		(property "Reference" "#PWR0143"
 			(at 97.79 179.07 0)
 			(effects
@@
 			(project "frothfet"
 				(path "/c83c6236-96e9-46ad-9d7a-9e2efa4a7966/777fe0ac-daa5-4cfe-9bd1-5eba0a425019"
-					(reference "#PWR0141")
+					(reference "#PWR0143")
 					(unit 1)
 				)
@@
 		(on_board yes)
 		(dnp no)
-		(property "Reference" "#PWR0153"
+		(property "Reference" "#PWR0155"
 			(at 220.98 119.38 0)
 			(effects
@@
 			(project "frothfet"
 				(path "/c83c6236-96e9-46ad-9d7a-9e2efa4a7966/777fe0ac-daa5-4cfe-9bd1-5eba0a425019"
-					(reference "#PWR0153")
+					(reference "#PWR0155")
 					(unit 1)
 				)
@@
 		(dnp no)
 		(fields_autoplaced yes)
-		(property "Reference" "#PWR0145"
+		(property "Reference" "#PWR0147"
 			(at 115.57 81.28 0)
 			(effects
@@
 			(project "frothfet"
 				(path "/c83c6236-96e9-46ad-9d7a-9e2efa4a7966/777fe0ac-daa5-4cfe-9bd1-5eba0a425019"
-					(reference "#PWR0145")
+					(reference "#PWR0147")
 					(unit 1)
 				)
@@
 		(on_board yes)
 		(dnp no)
-		(property "Reference" "#PWR0147"
+		(property "Reference" "#PWR0149"
 			(at 163.83 31.75 0)
 			(effects
@@
 			(project "frothfet"
 				(path "/c83c6236-96e9-46ad-9d7a-9e2efa4a7966/777fe0ac-daa5-4cfe-9bd1-5eba0a425019"
-					(reference "#PWR0147")
+					(reference "#PWR0149")
 					(unit 1)
 				)
@@
 		(on_board yes)
 		(dnp no)
-		(property "Reference" "#PWR0152"
+		(property "Reference" "#PWR0154"
 			(at 213.36 64.77 0)
 			(effects
@@
 			(project "frothfet"
 				(path "/c83c6236-96e9-46ad-9d7a-9e2efa4a7966/777fe0ac-daa5-4cfe-9bd1-5eba0a425019"
-					(reference "#PWR0152")
+					(reference "#PWR0154")
 					(unit 1)
 				)
@@
 		(dnp yes)
 		(fields_autoplaced yes)
-		(property "Reference" "J13"
+		(property "Reference" "J14"
 			(at 121.92 179.0699 0)
 			(effects
@@
 			(project "frothfet"
 				(path "/c83c6236-96e9-46ad-9d7a-9e2efa4a7966/777fe0ac-daa5-4cfe-9bd1-5eba0a425019"
-					(reference "J13")
+					(reference "J14")
 					(unit 1)
 				)
@@
 		(on_board yes)
 		(dnp no)
-		(property "Reference" "#PWR0148"
+		(property "Reference" "#PWR0150"
 			(at 184.15 119.38 0)
 			(effects
@@
 			(project "frothfet"
 				(path "/c83c6236-96e9-46ad-9d7a-9e2efa4a7966/777fe0ac-daa5-4cfe-9bd1-5eba0a425019"
-					(reference "#PWR0148")
+					(reference "#PWR0150")
 					(unit 1)
 				)
@@
 		(dnp no)
 		(fields_autoplaced yes)
-		(property "Reference" "#PWR0142"
+		(property "Reference" "#PWR0144"
 			(at 97.79 186.69 0)
 			(effects
@@
 			(project "frothfet"
 				(path "/c83c6236-96e9-46ad-9d7a-9e2efa4a7966/777fe0ac-daa5-4cfe-9bd1-5eba0a425019"
-					(reference "#PWR0142")
+					(reference "#PWR0144")
 					(unit 1)
 				)
@@
 		(dnp no)
 		(fields_autoplaced yes)
-		(property "Reference" "#PWR0140"
+		(property "Reference" "#PWR0142"
 			(at 85.09 162.56 0)
 			(effects
@@
 			(project "frothfet"
 				(path "/c83c6236-96e9-46ad-9d7a-9e2efa4a7966/777fe0ac-daa5-4cfe-9bd1-5eba0a425019"
-					(reference "#PWR0140")
+					(reference "#PWR0142")
 					(unit 1)
 				)
@@
 		(dnp no)
 		(fields_autoplaced yes)
-		(property "Reference" "#PWR0151"
+		(property "Reference" "#PWR0153"
 			(at 204.47 83.82 0)
 			(effects
@@
 			(project "frothfet"
 				(path "/c83c6236-96e9-46ad-9d7a-9e2efa4a7966/777fe0ac-daa5-4cfe-9bd1-5eba0a425019"
-					(reference "#PWR0151")
+					(reference "#PWR0153")
 					(unit 1)
 				)
@@
 		(dnp no)
 		(fields_autoplaced yes)
-		(property "Reference" "#PWR0155"
+		(property "Reference" "#PWR0157"
 			(at 229.87 144.78 0)
 			(effects
@@
 			(project "frothfet"
 				(path "/c83c6236-96e9-46ad-9d7a-9e2efa4a7966/777fe0ac-daa5-4cfe-9bd1-5eba0a425019"
-					(reference "#PWR0155")
+					(reference "#PWR0157")
 					(unit 1)
 				)
@@
 		(dnp no)
 		(fields_autoplaced yes)
-		(property "Reference" "#PWR0149"
+		(property "Reference" "#PWR0151"
 			(at 193.04 143.51 0)
 			(effects
@@
 			(project "frothfet"
 				(path "/c83c6236-96e9-46ad-9d7a-9e2efa4a7966/777fe0ac-daa5-4cfe-9bd1-5eba0a425019"
-					(reference "#PWR0149")
+					(reference "#PWR0151")
 					(unit 1)
 				)
@@
 		(dnp no)
 		(fields_autoplaced yes)
-		(property "Reference" "#PWR0144"
+		(property "Reference" "#PWR0146"
 			(at 109.22 48.26 0)
 			(effects
@@
 			(project "frothfet"
 				(path "/c83c6236-96e9-46ad-9d7a-9e2efa4a7966/777fe0ac-daa5-4cfe-9bd1-5eba0a425019"
-					(reference "#PWR0144")
+					(reference "#PWR0146")
 					(unit 1)
 				)
@@
 		(on_board yes)
 		(dnp no)
-		(property "Reference" "#PWR0143"
+		(property "Reference" "#PWR0145"
 			(at 106.68 100.33 0)
 			(effects
@@
 			(project "frothfet"
 				(path "/c83c6236-96e9-46ad-9d7a-9e2efa4a7966/777fe0ac-daa5-4cfe-9bd1-5eba0a425019"
-					(reference "#PWR0143")
+					(reference "#PWR0145")
 					(unit 1)
 				)
@@
 		(dnp no)
 		(fields_autoplaced yes)
-		(property "Reference" "J12"
+		(property "Reference" "J13"
 			(at 68.58 27.94 0)
 			(effects
@@
 			(project "frothfet"
 				(path "/c83c6236-96e9-46ad-9d7a-9e2efa4a7966/777fe0ac-daa5-4cfe-9bd1-5eba0a425019"
-					(reference "J12")
+					(reference "J13")
 					(unit 1)
 				)
@@
 		(on_board yes)
 		(dnp no)
-		(property "Reference" "#PWR0154"
+		(property "Reference" "#PWR0156"
 			(at 224.79 31.75 0)
 			(effects
@@
 			(project "frothfet"
 				(path "/c83c6236-96e9-46ad-9d7a-9e2efa4a7966/777fe0ac-daa5-4cfe-9bd1-5eba0a425019"
-					(reference "#PWR0154")
+					(reference "#PWR0156")
 					(unit 1)
 				)
@@
 		(dnp no)
 		(fields_autoplaced yes)
-		(property "Reference" "#PWR0139"
+		(property "Reference" "#PWR0141"
 			(at 64.77 80.01 0)
 			(effects
@@
 			(project "frothfet"
 				(path "/c83c6236-96e9-46ad-9d7a-9e2efa4a7966/777fe0ac-daa5-4cfe-9bd1-5eba0a425019"
-					(reference "#PWR0139")
+					(reference "#PWR0141")
 					(unit 1)
 				)
@@
 		(on_board yes)
 		(dnp no)
-		(property "Reference" "#PWR0146"
+		(property "Reference" "#PWR0148"
 			(at 125.73 36.83 0)
 			(effects
@@
 			(project "frothfet"
 				(path "/c83c6236-96e9-46ad-9d7a-9e2efa4a7966/777fe0ac-daa5-4cfe-9bd1-5eba0a425019"
-					(reference "#PWR0146")
+					(reference "#PWR0148")
 					(unit 1)
 				)
@@
 		(dnp no)
 		(fields_autoplaced yes)
-		(property "Reference" "#PWR0150"
+		(property "Reference" "#PWR0152"
 			(at 198.12 48.26 0)
 			(effects
@@
 			(project "frothfet"
 				(path "/c83c6236-96e9-46ad-9d7a-9e2efa4a7966/777fe0ac-daa5-4cfe-9bd1-5eba0a425019"
-					(reference "#PWR0150")
+					(reference "#PWR0152")
 					(unit 1)
 				)

Commit message: silkscreen and 3d models complete
Parts:
- J14: now fitted
Changed lines of the file:
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@@
 		(in_bom yes)
 		(on_board yes)
-		(dnp yes)
+		(dnp no)
 		(fields_autoplaced yes)
 		(property "Reference" "J14"

Commit message: added some lcsc part numbers
Parts:
- J14: LCSC (none) -> C780062
Changed lines of the file:
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@@
+			)
+		)
+		(property "LCSC" "C780062"
+			(at 119.38 179.07 0)
+			(effects
+				(font
+					(size 1.27 1.27)
+				)
+				(hide yes)
 			)
 		)

Commit message: added more esd protection to 3.3v and 5v rails.
Parts:
- removed D37: GREEN, LED_SMD:LED_0603_1608Metric, symbol Device:LED
- removed R56: 5.1k, Resistor_SMD:R_0603_1608Metric, symbol Device:R_Small_US
- added D39: SMAJ3.3A, Diode_SMD:D_SMA, symbol Device:D_TVS
- J14: LCSC C780062 -> (none); now not fitted
- renumbered D35 to D37, D36 to D38, R52 to R53, R53 to R54, R54 to R55, R55 to R56, TP27 to TP26, TP26 to TP27
Connections:
- net +3.3V: now also D39.2 (A2)
- net GND: now also D39.1 (A1)
Other:
- company: https://github.com/hoeken/frothfet -> (none)
- title: FrothFET 8CH -> https://github.com/hoeken/brineomatic
- moved on the sheet: C68, C70, TP27, U33
