File: frothfet/esp32-s3.kicad_sch (KiCad schematic)
At the start: 29 parts, among them J4 USB_TYPE_C_16PIN, J5 Conn_01x04, SW1 BOOT, SW2 RESET, U30 ESP32-S3-WROOM-1-N16R8, U31 USBLC6-2SC6, U32 SN74LV1T34DBV, U33 XC6210B332MR

Commit message: pulled in latest version of esp32 schematic
Parts:
- removed C64: 10uF, Capacitor_SMD:C_0603_1608Metric, symbol Device:C_Small
- removed C68: 1uF, Capacitor_SMD:C_0603_1608Metric, symbol Device:C_Small
- removed U33: XC6210B332MR, Package_TO_SOT_SMD:SOT-23-5, symbol Regulator_Linear:XC6210B332MR
- added D48: GREEN, LED_SMD:LED_0603_1608Metric, symbol Device:LED
- added R65: 5.1k, Resistor_SMD:R_0603_1608Metric, symbol Device:R_Small_US
- added U32: LDL1117S33R, Package_TO_SOT_SMD:SOT-223-3_TabPin2, symbol Regulator_Linear:AMS1117-3.3
- C67: renamed from C70; value 10uF -> 4.7uF
- D45: value SS36 -> SS34; LCSC C16015 -> C8678
- J5: footprint Connector_PinHeader_2.54mm:PinHeader_1x04_P2.54mm_Vertical_SMD_Pin1Right -> Connector_PinHeader_2.54mm:PinHeader_1x04_P2.54mm_Vertical_SMD_Pin1Left; now not fitted
- SW1: value BOOT -> ~
- SW2: value RESET -> ~
- renumbered C65 to C64, C66 to C65, C67 to C66, C69 to C68, C71 to C69, TP43 to TP42, TP42 to TP43, U32 to U33
Connections:
- net +3.3V: now also D48.2 (A), U32.2 (VO)
- net +5V: now also U32.3 (VI)
- net GND: now also R65.2, U32.1 (GND)
- new net: D48.1 (K), R65.1
Other:
- note added: "BOOT"
- note added: "RESET"
- moved on the sheet: C65, C67, D47, TP42

Commit message: updated bom and checked placement
Parts:
- D48: LCSC (none) -> C12624
- R61, R62, R65: LCSC (none) -> C23186
- R63, R64: LCSC (none) -> C25804
Changed lines of the file:
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@@
 			)
 		)
-		(property "LCSC" ""
+		(property "LCSC" "C23186"
 			(at 99.06 43.18 90)
 			(effects
@@
 			)
 		)
-		(property "LCSC" ""
+		(property "LCSC" "C12624"
 			(at 233.68 34.29 90)
 			(effects
@@
 			)
 		)
+		(property "LCSC" "C25804"
+			(at 184.15 119.38 0)
+			(effects
+				(font
+					(size 1.27 1.27)
+				)
+				(hide yes)
+			)
+		)
 		(pin "1"
 		)
@@
 			)
 		)
-		(property "LCSC" ""
+		(property "LCSC" "C23186"
 			(at 99.06 40.64 90)
 			(effects
@@
 			)
 		)
+		(property "LCSC" "C23186"
+			(at 233.68 40.64 0)
+			(effects
+				(font
+					(size 1.27 1.27)
+				)
+				(hide yes)
+			)
+		)
 		(pin "1"
 		)
@@
 			(at 220.98 119.38 0)
 			(effects
+				(font
+					(size 1.27 1.27)
+				)
+				(hide yes)
+			)
+		)
+		(property "LCSC" "C25804"
+			(at 220.98 119.38 0)
+			(effects
